File: pcb-tacho/pcb-tacho.sch (KiCad schematic (older format))
At the start: 13 parts, among them J1 Conn_01x03_Male, U1 LM555xM

Commit message: started v1.1
Parts:
- removed C1: 100n, Capacitor_SMD:C_1206_3216Metric_Pad1.33x1.80mm_HandSolder, symbol Device:C
- removed R4: 47k, Resistor_SMD:R_1206_3216Metric_Pad1.30x1.75mm_HandSolder, symbol Device:R
- added U2: TachoCapPlate, footprints:TachoCapPlate, symbol symbols:TachoCapPlate
Connections:
- net at R1.1: now also U2.~
Other:
- moved on the sheet: D1, D3, R1
Changed lines of the file:
@@
 $EndDescr
-$Comp
-L Device:C C1
-U 1 1 616A80FF
-P 3650 3250
-F 0 "C1" V 3800 3250 50  0000 C CNN
-F 1 "100n" V 3489 3250 50  0000 C CNN
-F 2 "Capacitor_SMD:C_1206_3216Metric_Pad1.33x1.80mm_HandSolder" H 3688 3100 50  0001 C CNN
-F 3 "~" H 3650 3250 50  0001 C CNN
-	1    3650 3250
-	-1   0    0    1
-$EndComp
 $Comp
 L Device:R R1
 U 1 1 616A8BBE
-P 2900 3000
-F 0 "R1" V 3107 3000 50  0000 C CNN
-F 1 "1k" V 3016 3000 50  0000 C CNN
-F 2 "Resistor_SMD:R_1206_3216Metric_Pad1.30x1.75mm_HandSolder" V 2830 3000 50  0001 C CNN
-F 3 "~" H 2900 3000 50  0001 C CNN
-	1    2900 3000
+P 3600 3000
+F 0 "R1" V 3807 3000 50  0000 C CNN
+F 1 "1k" V 3716 3000 50  0000 C CNN
+F 2 "Resistor_SMD:R_1206_3216Metric_Pad1.30x1.75mm_HandSolder" V 3530 3000 50  0001 C CNN
+F 3 "~" H 3600 3000 50  0001 C CNN
+	1    3600 3000
 	0    -1   -1   0
 $EndComp
@@
 L Device:D_Zener D1
 U 1 1 616A9652
-P 3150 3250
-F 0 "D1" V 3104 3330 50  0000 L CNN
-F 1 "5V" V 3195 3330 50  0000 L CNN
-F 2 "Diode_SMD:D_1206_3216Metric_Pad1.42x1.75mm_HandSolder" H 3150 3250 50  0001 C CNN
-F 3 "~" H 3150 3250 50  0001 C CNN
-	1    3150 3250
+P 3850 3250
+F 0 "D1" V 3804 3330 50  0000 L CNN
+F 1 "5V" V 3895 3330 50  0000 L CNN
+F 2 "Diode_SMD:D_1206_3216Metric_Pad1.42x1.75mm_HandSolder" H 3850 3250 50  0001 C CNN
+F 3 "~" H 3850 3250 50  0001 C CNN
+	1    3850 3250
 	0    1    1    0
 $EndComp
@@
 L power:GND #PWR01
 U 1 1 616A9D72
-P 3150 3500
-F 0 "#PWR01" H 3150 3250 50  0001 C CNN
-F 1 "GND" H 3155 3327 50  0000 C CNN
-F 2 "" H 3150 3500 50  0001 C CNN
-F 3 "" H 3150 3500 50  0001 C CNN
-	1    3150 3500
+P 3850 3500
+F 0 "#PWR01" H 3850 3250 50  0001 C CNN
+F 1 "GND" H 3855 3327 50  0000 C CNN
+F 2 "" H 3850 3500 50  0001 C CNN
+F 3 "" H 3850 3500 50  0001 C CNN
+	1    3850 3500
 	1    0    0    -1
 $EndComp
@@
 $EndComp
 $Comp
-L power:GND #PWR014
-U 1 1 616CEF73
-P 3650 3500
-F 0 "#PWR014" H 3650 3250 50  0001 C CNN
-F 1 "GND" H 3655 3327 50  0000 C CNN
-F 2 "" H 3650 3500 50  0001 C CNN
-F 3 "" H 3650 3500 50  0001 C CNN
-	1    3650 3500
-	1    0    0    -1
-$EndComp
-$Comp
 L Timer:LM555xM U1
 U 1 1 616E1136
@@
 L Device:D D3
 U 1 1 616F189C
-P 3400 3000
-F 0 "D3" H 3400 2783 50  0000 C CNN
-F 1 "D" H 3400 2874 50  0000 C CNN
-F 2 "Diode_SMD:D_1206_3216Metric_Pad1.42x1.75mm_HandSolder" H 3400 3000 50  0001 C CNN
-F 3 "~" H 3400 3000 50  0001 C CNN
-	1    3400 3000
+P 4100 3000
+F 0 "D3" H 4100 2783 50  0000 C CNN
+F 1 "D" H 4100 2874 50  0000 C CNN
+F 2 "Diode_SMD:D_1206_3216Metric_Pad1.42x1.75mm_HandSolder" H 4100 3000 50  0001 C CNN
+F 3 "~" H 4100 3000 50  0001 C CNN
+	1    4100 3000
 	-1   0    0    1
 $EndComp
-$Comp
-L Device:R R4
-U 1 1 616F1F09
-P 4000 3250
-F 0 "R4" H 4070 3296 50  0000 L CNN
-F 1 "47k" H 4070 3205 50  0000 L CNN
-F 2 "Resistor_SMD:R_1206_3216Metric_Pad1.30x1.75mm_HandSolder" V 3930 3250 50  0001 C CNN
-F 3 "~" H 4000 3250 50  0001 C CNN
-	1    4000 3250
-	1    0    0    -1
-$EndComp
-Wire Wire Line
-	3050 3000 3150 3000
-Wire Wire Line
-	3150 3000 3150 3100
-Connection ~ 3150 3000
-Wire Wire Line
-	3150 3000 3250 3000
-Wire Wire Line
-	3150 3400 3150 3500
-Wire Wire Line
-	3650 3500 3650 3400
-Wire Wire Line
-	3550 3000 3650 3000
-Wire Wire Line
-	3650 3000 3650 3100
-Wire Wire Line
-	4000 3000 4000 3100
-$Comp
-L power:GND #PWR013
-U 1 1 6170CCE6
-P 4000 3500
-F 0 "#PWR013" H 4000 3250 50  0001 C CNN
-F 1 "GND" H 4005 3327 50  0000 C CNN
-F 2 "" H 4000 3500 50  0001 C CNN
-F 3 "" H 4000 3500 50  0001 C CNN
-	1    4000 3500
-	1    0    0    -1
-$EndComp
-Wire Wire Line
-	4000 3500 4000 3400
-Wire Wire Line
-	4000 3000 4900 3000
+Wire Wire Line
+	3750 3000 3850 3000
+Wire Wire Line
+	3850 3000 3850 3100
+Connection ~ 3850 3000
+Wire Wire Line
+	3850 3000 3950 3000
+Wire Wire Line
+	3850 3400 3850 3500
 Wire Wire Line
 	4600 3400 4900 3400
@@
 	5400 3800 5400 3600
 Wire Wire Line
-	3650 3000 4000 3000
-Connection ~ 3650 3000
-Connection ~ 4000 3000
+	4250 3000 4900 3000
+$Comp
+L symbols:TachoCapPlate U2
+U 1 1 616C6105
+P 2700 3000
+F 0 "U2" H 2833 3265 50  0000 C CNN
+F 1 "TachoCapPlate" H 2833 3174 50  0000 C CNN
+F 2 "footprints:TachoCapPlate" H 2700 3000 50  0001 C CNN
+F 3 "" H 2700 3000 50  0001 C CNN
+	1    2700 3000
+	1    0    0    -1
+$EndComp
+Wire Wire Line
+	3350 3000 3450 3000
 $EndSCHEMATC

Commit message: more v1.1
Parts:
- C3: footprint Capacitor_SMD:CP_Elec_8x10 -> Capacitor_THT:CP_Radial_D10.0mm_P3.80mm
- U2: symbol symbols:TachoCapPlate -> pcb-tacho-rescue:TachoCapPlate-symbols
Other:
- moved on the sheet: C3, D2, R3
Changed lines of the file:
@@
 L Device:D_Zener D2
 U 1 1 616AA237
-P 7400 3300
-F 0 "D2" V 7354 3380 50  0000 L CNN
-F 1 "9V" V 7445 3380 50  0000 L CNN
-F 2 "Diode_SMD:D_1206_3216Metric_Pad1.42x1.75mm_HandSolder" H 7400 3300 50  0001 C CNN
-F 3 "~" H 7400 3300 50  0001 C CNN
-	1    7400 3300
+P 7600 2750
+F 0 "D2" V 7554 2830 50  0000 L CNN
+F 1 "9V" V 7645 2830 50  0000 L CNN
+F 2 "Diode_SMD:D_1206_3216Metric_Pad1.42x1.75mm_HandSolder" H 7600 2750 50  0001 C CNN
+F 3 "~" H 7600 2750 50  0001 C CNN
+	1    7600 2750
 	0    1    1    0
 $EndComp
@@
 L power:GND #PWR07
 U 1 1 616AA553
-P 7400 3650
-F 0 "#PWR07" H 7400 3400 50  0001 C CNN
-F 1 "GND" H 7405 3477 50  0000 C CNN
-F 2 "" H 7400 3650 50  0001 C CNN
-F 3 "" H 7400 3650 50  0001 C CNN
-	1    7400 3650
+P 7600 3100
+F 0 "#PWR07" H 7600 2850 50  0001 C CNN
+F 1 "GND" H 7605 2927 50  0000 C CNN
+F 2 "" H 7600 3100 50  0001 C CNN
+F 3 "" H 7600 3100 50  0001 C CNN
+	1    7600 3100
 	1    0    0    -1
 $EndComp
@@
 L power:+9V #PWR06
 U 1 1 616AAC57
-P 7400 2950
-F 0 "#PWR06" H 7400 2800 50  0001 C CNN
-F 1 "+9V" H 7415 3123 50  0000 C CNN
-F 2 "" H 7400 2950 50  0001 C CNN
-F 3 "" H 7400 2950 50  0001 C CNN
-	1    7400 2950
+P 7600 2400
+F 0 "#PWR06" H 7600 2250 50  0001 C CNN
+F 1 "+9V" H 7615 2573 50  0000 C CNN
+F 2 "" H 7600 2400 50  0001 C CNN
+F 3 "" H 7600 2400 50  0001 C CNN
+	1    7600 2400
 	1    0    0    -1
 $EndComp
@@
 L Device:R R3
 U 1 1 616B2568
-P 7650 3050
-F 0 "R3" V 7443 3050 50  0000 C CNN
-F 1 "15" V 7534 3050 50  0000 C CNN
-F 2 "Resistor_SMD:R_1206_3216Metric_Pad1.30x1.75mm_HandSolder" V 7580 3050 50  0001 C CNN
-F 3 "~" H 7650 3050 50  0001 C CNN
-	1    7650 3050
+P 7850 2500
+F 0 "R3" V 7643 2500 50  0000 C CNN
+F 1 "15" V 7734 2500 50  0000 C CNN
+F 2 "Resistor_SMD:R_1206_3216Metric_Pad1.30x1.75mm_HandSolder" V 7780 2500 50  0001 C CNN
+F 3 "~" H 7850 2500 50  0001 C CNN
+	1    7850 2500
 	0    1    1    0
 $EndComp
@@
 L power:+12V #PWR08
 U 1 1 616B2DA0
-P 7900 2950
-F 0 "#PWR08" H 7900 2800 50  0001 C CNN
-F 1 "+12V" H 7915 3123 50  0000 C CNN
-F 2 "" H 7900 2950 50  0001 C CNN
-F 3 "" H 7900 2950 50  0001 C CNN
-	1    7900 2950
+P 8100 2400
+F 0 "#PWR08" H 8100 2250 50  0001 C CNN
+F 1 "+12V" H 8115 2573 50  0000 C CNN
+F 2 "" H 8100 2400 50  0001 C CNN
+F 3 "" H 8100 2400 50  0001 C CNN
+	1    8100 2400
 	1    0    0    -1
 $EndComp
@@
 L Device:CP C3
 U 1 1 616B42F3
-P 7050 3300
-F 0 "C3" H 7168 3346 50  0000 L CNN
-F 1 "10u" H 7168 3255 50  0000 L CNN
-F 2 "Capacitor_SMD:CP_Elec_8x10" H 7088 3150 50  0001 C CNN
-F 3 "~" H 7050 3300 50  0001 C CNN
-	1    7050 3300
+P 7250 2750
+F 0 "C3" H 7368 2796 50  0000 L CNN
+F 1 "10u" H 7368 2705 50  0000 L CNN
+F 2 "Capacitor_THT:CP_Radial_D10.0mm_P3.80mm" H 7288 2600 50  0001 C CNN
+F 3 "~" H 7250 2750 50  0001 C CNN
+	1    7250 2750
 	1    0    0    -1
 $EndComp
@@
 	4600 3400 4900 3400
 Wire Wire Line
-	7500 3050 7400 3050
-Wire Wire Line
-	7050 3050 7050 3150
-Wire Wire Line
-	7400 3150 7400 3050
-Connection ~ 7400 3050
-Wire Wire Line
-	7400 3050 7050 3050
-Wire Wire Line
-	7400 3050 7400 2950
-Wire Wire Line
-	7400 3450 7400 3550
-Wire Wire Line
-	7400 3550 7050 3550
-Wire Wire Line
-	7050 3550 7050 3450
-Connection ~ 7400 3550
-Wire Wire Line
-	7400 3550 7400 3650
-Wire Wire Line
-	7800 3050 7900 3050
-Wire Wire Line
-	7900 3050 7900 2950
+	7700 2500 7600 2500
+Wire Wire Line
+	7250 2500 7250 2600
+Wire Wire Line
+	7600 2600 7600 2500
+Connection ~ 7600 2500
+Wire Wire Line
+	7600 2500 7250 2500
+Wire Wire Line
+	7600 2500 7600 2400
+Wire Wire Line
+	7600 2900 7600 3000
+Wire Wire Line
+	7600 3000 7250 3000
+Wire Wire Line
+	7250 3000 7250 2900
+Connection ~ 7600 3000
+Wire Wire Line
+	7600 3000 7600 3100
+Wire Wire Line
+	8000 2500 8100 2500
+Wire Wire Line
+	8100 2500 8100 2400
 Wire Wire Line
 	5900 3400 6000 3400
@@
 	4250 3000 4900 3000
 $Comp
-L symbols:TachoCapPlate U2
+L pcb-tacho-rescue:TachoCapPlate-symbols U2
 U 1 1 616C6105
 P 2700 3000
