File: pcb-tacho/pcb-tacho.kicad_pcb (KiCad board)
At the start: 2 copper layers, 42 x 39 mm, 12 parts, among them J1 Conn_01x03_Male, U1 LM555xM, U2 TachoCapPlate

Commit message: more v1.1
Parts:
- C3: footprint Capacitor_SMD:CP_Elec_8x10 -> Capacitor_THT:CP_Radial_D10.0mm_P3.80mm
Connections:
- U2 pad 1: Net-(R1-Pad1) -> (no net)

Commit message: tacho sensor pcb
Parts:
- moved C4 19.5 mm to (145.0, 82.4), turned to 90 degrees
- moved D2 12.4 mm to (160.5, 98.4)
- moved R2 2.96 mm to (150.0, 87.5), turned to -90 degrees
- moved C2 2.83 mm to (150.0, 92.6), turned to 90 degrees
- moved U1 2.65 mm to (142.6, 89.7), turned to 90 degrees
Other:
- net class Default removed
