File: pcb-main/pcb-main.sch (KiCad schematic (older format))
At the start: 26 parts, among them J1 AVR-ISP-6, M1 Stepper_Motor, U1 ATmega328P-AU, U2 HT1621B, U3 VIM878, U4 MC7805CD

Commit message: lcd and mcu
Parts:
- added R7: 10k, symbol Device:R
- J1: footprint Connector_PinSocket_2.54mm:PinSocket_2x03_P2.54mm_Vertical_SMD -> Connector_PinHeader_2.54mm:PinHeader_2x03_P2.54mm_Vertical_SMD
Connections:
- wire segments 66 -> 70
Changed lines of the file:
@@
 F 0 "J1" H 3771 1596 50  0000 R CNN
 F 1 "AVR-ISP-6" H 3771 1505 50  0000 R CNN
-F 2 "Connector_PinSocket_2.54mm:PinSocket_2x03_P2.54mm_Vertical_SMD" V 3850 1550 50  0001 C CNN
+F 2 "Connector_PinHeader_2.54mm:PinHeader_2x03_P2.54mm_Vertical_SMD" V 3850 1550 50  0001 C CNN
 F 3 " ~" H 2825 950 50  0001 C CNN
 	1    4100 1500
@@
 Text Label 4500 1600 0    50   ~ 0
 RESET
-Text Label 2650 2900 0    50   ~ 0
+Text Label 3400 2900 0    50   ~ 0
 RESET
 $Comp
@@
 Text Label 1600 6300 2    50   ~ 0
 LCD_DATA
-Text Label 2650 1400 0    50   ~ 0
+Text Label 2950 1700 0    50   ~ 0
 LCD_CS
-Text Label 2650 1500 0    50   ~ 0
+Text Label 2950 1800 0    50   ~ 0
 LCD_WR
-Text Label 2650 1600 0    50   ~ 0
+Text Label 2950 1900 0    50   ~ 0
 LCD_DATA
 Text Notes 3550 4350 0    50   ~ 0
@@
 	5750 3150 5850 3150
 $Comp
-L power:GND #PWR?
+L power:GND #PWR0113
 U 1 1 6149D2EC
 P 5750 3650
-F 0 "#PWR?" H 5750 3400 50  0001 C CNN
+F 0 "#PWR0113" H 5750 3400 50  0001 C CNN
 F 1 "GND" H 5755 3477 50  0000 C CNN
 F 2 "" H 5750 3650 50  0001 C CNN
@@
 Text Label 7100 2200 0    50   ~ 0
 SPEEDO
+$Comp
+L power:+5V #PWR?
+U 1 1 613D3197
+P 3250 2400
+AR Path="/612034A3/613D3197" Ref="#PWR?"  Part="1"
+AR Path="/613D3197" Ref="#PWR0114"  Part="1"
+F 0 "#PWR0114" H 3250 2250 50  0001 C CNN
+F 1 "+5V" H 3265 2573 50  0000 C CNN
+F 2 "" H 3250 2400 50  0001 C CNN
+F 3 "" H 3250 2400 50  0001 C CNN
+	1    3250 2400
+	1    0    0    -1
+$EndComp
+$Comp
+L Device:R R7
+U 1 1 613D3AC3
+P 3250 2650
+F 0 "R7" H 3180 2604 50  0000 R CNN
+F 1 "10k" H 3180 2695 50  0000 R CNN
+F 2 "" V 3180 2650 50  0001 C CNN
+F 3 "~" H 3250 2650 50  0001 C CNN
+	1    3250 2650
+	-1   0    0    1
+$EndComp
+Wire Wire Line
+	3400 2900 3250 2900
+Wire Wire Line
+	3250 2800 3250 2900
+Connection ~ 3250 2900
+Wire Wire Line
+	3250 2900 2650 2900
+Wire Wire Line
+	3250 2500 3250 2400
 $EndSCHEMATC

Commit message: added stepper motor spike (and heaps of other stuff)
Parts:
- removed D10, D12, D13, D9: LED, LED_SMD:LED_1206_3216Metric_Pad1.42x1.75mm_HandSolder, symbol Device:LED
- removed R1, R2, R4, R5: R, Resistor_SMD:R_1206_3216Metric_Pad1.30x1.75mm_HandSolder, symbol Device:R
- removed U4: MC7805CD, symbol symbols:MC7805CD
- added C1, C2, C3, C4: C, Capacitor_SMD:C_1206_3216Metric_Pad1.33x1.80mm_HandSolder, symbol Device:C
- added J2: Conn_02x06_Counter_Clockwise, Connector_PinHeader_2.54mm:PinHeader_2x06_P2.54mm_Vertical_SMD, symbol Connector_Generic:Conn_02x06_Counter_Clockwise
- added J3: Conn_02x02_Counter_Clockwise, Connector_PinHeader_2.54mm:PinHeader_2x02_P2.54mm_Vertical_SMD, symbol Connector_Generic:Conn_02x02_Counter_Clockwise
- added SW?: SW_Push, symbol Switch:SW_Push
- added Y1: Crystal, Crystal:Crystal_HC49-4H_Vertical, symbol Device:Crystal
- D11, D14: value LED -> BACKLIGHT
- J1: footprint Connector_PinHeader_2.54mm:PinHeader_2x03_P2.54mm_Vertical_SMD -> Connector_PinHeader_2.54mm:PinHeader_2x03_P2.54mm_Vertical
- R7: footprint (none) -> Resistor_SMD:R_1206_3216Metric_Pad1.30x1.75mm_HandSolder
- U2: footprint Package_SO:SSOP-48_7.5x15.9mm_P0.635mm -> footprints:HT1621B
Connections:
- net labels added: ADC6, ADC7, BACKLIGHT_LED, MOT_1, MOT_2, MOT_3, MOT_4, PB0, PB3, PB4, PB5, PD0, PD1, PD2, PD3, PD4, PD5, PD6, PD7, XTAL1, XTAL2
- net labels removed: +12V, BATTERY_VOLTAGE, HIGH_BEAM, LCD_CS, LCD_DATA, LCD_WR, MISO, MOSI, MOT1, MOT2, MOT3, MOT4, NEUTRAL, OIL_PRESSURE, SCK, SPEEDO, TACHO, TURN_SIGNALS
- wire segments 70 -> 82
Other:
- note added: "Clock"
- note added: "ISP"
- note added: "LCD"
- note added: "TODO: change the footprint"
- note removed: "Power Supply"
- note removed: "TODO: Add connector to sensor PCB"
- note removed: "TODO: Clock battery backup"
- note removed: "TODO: Create the correct footprint for the power supply"
- note removed: "TODO: Double check all the pins"
- note removed: "TODO: Switch this from the MCU"
- note removed: "TODO: This is the wrong footprint"
- moved on the sheet: D11, D14, J1, R3, R6, U2, U3

Commit message: cleaned up main pcb
Parts:
- removed SW?: SW_Push, symbol Switch:SW_Push
- added U4: TLSM, footprints:TLSM, symbol symbols:TLSM
Connections:
- wire segments 82 -> 86
Other:
- note removed: "TODO: change the footprint"
- moved on the sheet: J1, J3
Changed lines of the file:
@@
 L power:+5V #PWR?
 U 1 1 612E399D
-P 4400 1050
+P 7300 4650
 AR Path="/612034A3/612E399D" Ref="#PWR?"  Part="1"
 AR Path="/612E399D" Ref="#PWR0104"  Part="1"
-F 0 "#PWR0104" H 4400 900 50  0001 C CNN
-F 1 "+5V" H 4415 1223 50  0000 C CNN
-F 2 "" H 4400 1050 50  0001 C CNN
-F 3 "" H 4400 1050 50  0001 C CNN
-	1    4400 1050
+F 0 "#PWR0104" H 7300 4500 50  0001 C CNN
+F 1 "+5V" H 7315 4823 50  0000 C CNN
+F 2 "" H 7300 4650 50  0001 C CNN
+F 3 "" H 7300 4650 50  0001 C CNN
+	1    7300 4650
 	1    0    0    -1
 $EndComp
@@
 L power:GND #PWR?
 U 1 1 612E39A4
-P 4400 2150
+P 7300 5750
 AR Path="/612034A3/612E39A4" Ref="#PWR?"  Part="1"
 AR Path="/612E39A4" Ref="#PWR0105"  Part="1"
-F 0 "#PWR0105" H 4400 1900 50  0001 C CNN
-F 1 "GND" H 4405 1977 50  0000 C CNN
-F 2 "" H 4400 2150 50  0001 C CNN
-F 3 "" H 4400 2150 50  0001 C CNN
-	1    4400 2150
+F 0 "#PWR0105" H 7300 5500 50  0001 C CNN
+F 1 "GND" H 7305 5577 50  0000 C CNN
+F 2 "" H 7300 5750 50  0001 C CNN
+F 3 "" H 7300 5750 50  0001 C CNN
+	1    7300 5750
 	1    0    0    -1
 $EndComp
@@
 L Connector:AVR-ISP-6 J?
 U 1 1 612E39AB
-P 4500 1650
+P 7400 5250
 AR Path="/612034A3/612E39AB" Ref="J?"  Part="1"
 AR Path="/612E39AB" Ref="J1"  Part="1"
-F 0 "J1" H 4171 1746 50  0000 R CNN
-F 1 "AVR-ISP-6" H 4171 1655 50  0000 R CNN
-F 2 "Connector_PinHeader_2.54mm:PinHeader_2x03_P2.54mm_Vertical" V 4250 1700 50  0001 C CNN
-F 3 " ~" H 3225 1100 50  0001 C CNN
-	1    4500 1650
-	1    0    0    -1
-$EndComp
-Text Label 4900 1550 0    50   ~ 0
+F 0 "J1" H 7071 5346 50  0000 R CNN
+F 1 "AVR-ISP-6" H 7071 5255 50  0000 R CNN
+F 2 "Connector_PinHeader_2.54mm:PinHeader_2x03_P2.54mm_Vertical" V 7150 5300 50  0001 C CNN
+F 3 " ~" H 6125 4700 50  0001 C CNN
+	1    7400 5250
+	1    0    0    -1
+$EndComp
+Text Label 7800 5150 0    50   ~ 0
 PB3
-Text Label 4900 1450 0    50   ~ 0
+Text Label 7800 5050 0    50   ~ 0
 PB4
-Text Label 4900 1650 0    50   ~ 0
+Text Label 7800 5250 0    50   ~ 0
 PB5
-Text Label 4900 1750 0    50   ~ 0
+Text Label 7800 5350 0    50   ~ 0
 RESET
 Text Label 3400 2900 0    50   ~ 0
@@
 Connection ~ 2150 1000
 Wire Wire Line
-	4400 1050 4400 1150
-Wire Wire Line
-	4400 2050 4400 2150
+	7300 4650 7300 4750
+Wire Wire Line
+	7300 5650 7300 5750
 $Comp
 L Device:LED D11
@@
 Text Notes 2650 4900 0    50   ~ 0
 LCD
-Text Notes 4700 1050 0    50   ~ 0
+Text Notes 7600 4650 0    50   ~ 0
 ISP
 Wire Wire Line
@@
 L Connector_Generic:Conn_02x02_Counter_Clockwise J3
 U 1 1 61409762
-P 6850 2100
-F 0 "J3" H 6900 2317 50  0000 C CNN
-F 1 "Conn_02x02_Counter_Clockwise" H 6900 2226 50  0000 C CNN
-F 2 "Connector_PinHeader_2.54mm:PinHeader_2x02_P2.54mm_Vertical_SMD" H 6850 2100 50  0001 C CNN
-F 3 "~" H 6850 2100 50  0001 C CNN
-	1    6850 2100
+P 9500 5100
+F 0 "J3" H 9550 5317 50  0000 C CNN
+F 1 "Conn_02x02_Counter_Clockwise" H 9550 5226 50  0000 C CNN
+F 2 "Connector_PinHeader_2.54mm:PinHeader_2x02_P2.54mm_Vertical_SMD" H 9500 5100 50  0001 C CNN
+F 3 "~" H 9500 5100 50  0001 C CNN
+	1    9500 5100
 	1    0    0    -1
 $EndComp
 Text Label 2650 3100 0    50   ~ 0
 PD0
-Text Label 7250 2200 0    50   ~ 0
+Text Label 9900 5200 0    50   ~ 0
 PD0
 $Comp
 L power:+5V #PWR0112
 U 1 1 6140FFCF
-P 6550 2100
-F 0 "#PWR0112" H 6550 1950 50  0001 C CNN
-F 1 "+5V" V 6565 2228 50  0000 L CNN
-F 2 "" H 6550 2100 50  0001 C CNN
-F 3 "" H 6550 2100 50  0001 C CNN
-	1    6550 2100
+P 9200 5100
+F 0 "#PWR0112" H 9200 4950 50  0001 C CNN
+F 1 "+5V" V 9215 5228 50  0000 L CNN
+F 2 "" H 9200 5100 50  0001 C CNN
+F 3 "" H 9200 5100 50  0001 C CNN
+	1    9200 5100
 	0    -1   -1   0
 $EndComp
@@
 L power:GND #PWR0113
 U 1 1 614106F8
-P 6550 2300
-F 0 "#PWR0113" H 6550 2050 50  0001 C CNN
-F 1 "GND" H 6555 2127 50  0000 C CNN
-F 2 "" H 6550 2300 50  0001 C CNN
-F 3 "" H 6550 2300 50  0001 C CNN
-	1    6550 2300
-	1    0    0    -1
-$EndComp
-Wire Wire Line
-	7250 2200 7150 2200
-Wire Wire Line
-	6650 2100 6550 2100
-Wire Wire Line
-	6550 2300 6550 2200
-Wire Wire Line
-	6550 2200 6650 2200
-Text Notes 1150 4750 0    50   ~ 0
-TODO: change the footprint
-$Comp
-L Switch:SW_Push SW?
-U 1 1 615419CF
-P 4000 2900
-F 0 "SW?" H 4000 3185 50  0000 C CNN
-F 1 "SW_Push" H 4000 3094 50  0000 C CNN
-F 2 "" H 4000 3100 50  0001 C CNN
-F 3 "~" H 4000 3100 50  0001 C CNN
-	1    4000 2900
-	1    0    0    -1
-$EndComp
+P 9200 5300
+F 0 "#PWR0113" H 9200 5050 50  0001 C CNN
+F 1 "GND" H 9205 5127 50  0000 C CNN
+F 2 "" H 9200 5300 50  0001 C CNN
+F 3 "" H 9200 5300 50  0001 C CNN
+	1    9200 5300
+	1    0    0    -1
+$EndComp
+Wire Wire Line
+	9900 5200 9800 5200
+Wire Wire Line
+	9300 5100 9200 5100
+Wire Wire Line
+	9200 5300 9200 5200
+Wire Wire Line
+	9200 5200 9300 5200
+$Comp
+L symbols:TLSM U4
+U 1 1 61493463
+P 5600 1500
+F 0 "U4" H 5625 2115 50  0000 C CNN
+F 1 "TLSM" H 5625 2024 50  0000 C CNN
+F 2 "footprints:TLSM" H 5600 1500 50  0001 C CNN
+F 3 "" H 5600 1500 50  0001 C CNN
+	1    5600 1500
+	1    0    0    -1
+$EndComp
+Text Label 4950 1850 2    50   ~ 0
+RESET
+$Comp
+L power:GND #PWR0118
+U 1 1 6149B54A
+P 6400 1300
+F 0 "#PWR0118" H 6400 1050 50  0001 C CNN
+F 1 "GND" H 6405 1127 50  0000 C CNN
+F 2 "" H 6400 1300 50  0001 C CNN
+F 3 "" H 6400 1300 50  0001 C CNN
+	1    6400 1300
+	1    0    0    -1
+$EndComp
+Wire Wire Line
+	6300 1200 6400 1200
+Wire Wire Line
+	6400 1200 6400 1300
+$Comp
+L power:GND #PWR0119
+U 1 1 6149DF29
+P 4850 1300
+F 0 "#PWR0119" H 4850 1050 50  0001 C CNN
+F 1 "GND" H 4855 1127 50  0000 C CNN
+F 2 "" H 4850 1300 50  0001 C CNN
+F 3 "" H 4850 1300 50  0001 C CNN
+	1    4850 1300
+	1    0    0    -1
+$EndComp
+Wire Wire Line
+	4850 1300 4850 1200
+Wire Wire Line
+	4850 1200 4950 1200
 $EndSCHEMATC

Commit message: cleaned up main pcb
Connections:
- net GND: now also U4.3 (C), U4.4 (D)
- net RESET: now also U4.1 (A)
Other:
- moved on the sheet: J1, J3, U4
Changed lines of the file:
@@
 L power:+5V #PWR?
 U 1 1 612E399D
-P 7300 4650
+P 5950 1000
 AR Path="/612034A3/612E399D" Ref="#PWR?"  Part="1"
 AR Path="/612E399D" Ref="#PWR0104"  Part="1"
-F 0 "#PWR0104" H 7300 4500 50  0001 C CNN
-F 1 "+5V" H 7315 4823 50  0000 C CNN
-F 2 "" H 7300 4650 50  0001 C CNN
-F 3 "" H 7300 4650 50  0001 C CNN
-	1    7300 4650
+F 0 "#PWR0104" H 5950 850 50  0001 C CNN
+F 1 "+5V" H 5965 1173 50  0000 C CNN
+F 2 "" H 5950 1000 50  0001 C CNN
+F 3 "" H 5950 1000 50  0001 C CNN
+	1    5950 1000
 	1    0    0    -1
 $EndComp
@@
 L power:GND #PWR?
 U 1 1 612E39A4
-P 7300 5750
+P 5950 2100
 AR Path="/612034A3/612E39A4" Ref="#PWR?"  Part="1"
 AR Path="/612E39A4" Ref="#PWR0105"  Part="1"
-F 0 "#PWR0105" H 7300 5500 50  0001 C CNN
-F 1 "GND" H 7305 5577 50  0000 C CNN
-F 2 "" H 7300 5750 50  0001 C CNN
-F 3 "" H 7300 5750 50  0001 C CNN
-	1    7300 5750
+F 0 "#PWR0105" H 5950 1850 50  0001 C CNN
+F 1 "GND" H 5955 1927 50  0000 C CNN
+F 2 "" H 5950 2100 50  0001 C CNN
+F 3 "" H 5950 2100 50  0001 C CNN
+	1    5950 2100
 	1    0    0    -1
 $EndComp
@@
 L Connector:AVR-ISP-6 J?
 U 1 1 612E39AB
-P 7400 5250
+P 6050 1600
 AR Path="/612034A3/612E39AB" Ref="J?"  Part="1"
 AR Path="/612E39AB" Ref="J1"  Part="1"
-F 0 "J1" H 7071 5346 50  0000 R CNN
-F 1 "AVR-ISP-6" H 7071 5255 50  0000 R CNN
-F 2 "Connector_PinHeader_2.54mm:PinHeader_2x03_P2.54mm_Vertical" V 7150 5300 50  0001 C CNN
-F 3 " ~" H 6125 4700 50  0001 C CNN
-	1    7400 5250
-	1    0    0    -1
-$EndComp
-Text Label 7800 5150 0    50   ~ 0
+F 0 "J1" H 5721 1696 50  0000 R CNN
+F 1 "AVR-ISP-6" H 5721 1605 50  0000 R CNN
+F 2 "Connector_PinHeader_2.54mm:PinHeader_2x03_P2.54mm_Vertical" V 5800 1650 50  0001 C CNN
+F 3 " ~" H 4775 1050 50  0001 C CNN
+	1    6050 1600
+	1    0    0    -1
+$EndComp
+Text Label 6450 1500 0    50   ~ 0
 PB3
-Text Label 7800 5050 0    50   ~ 0
+Text Label 6450 1400 0    50   ~ 0
 PB4
-Text Label 7800 5250 0    50   ~ 0
+Text Label 6450 1600 0    50   ~ 0
 PB5
-Text Label 7800 5350 0    50   ~ 0
+Text Label 6450 1700 0    50   ~ 0
 RESET
 Text Label 3400 2900 0    50   ~ 0
@@
 Connection ~ 2150 1000
 Wire Wire Line
-	7300 4650 7300 4750
-Wire Wire Line
-	7300 5650 7300 5750
+	5950 1000 5950 1100
+Wire Wire Line
+	5950 2000 5950 2100
 $Comp
 L Device:LED D11
@@
 Text Notes 2650 4900 0    50   ~ 0
 LCD
-Text Notes 7600 4650 0    50   ~ 0
+Text Notes 6250 1000 0    50   ~ 0
 ISP
 Wire Wire Line
@@
 L Connector_Generic:Conn_02x02_Counter_Clockwise J3
 U 1 1 61409762
-P 9500 5100
-F 0 "J3" H 9550 5317 50  0000 C CNN
-F 1 "Conn_02x02_Counter_Clockwise" H 9550 5226 50  0000 C CNN
-F 2 "Connector_PinHeader_2.54mm:PinHeader_2x02_P2.54mm_Vertical_SMD" H 9500 5100 50  0001 C CNN
-F 3 "~" H 9500 5100 50  0001 C CNN
-	1    9500 5100
+P 8700 3550
+F 0 "J3" H 8750 3767 50  0000 C CNN
+F 1 "Conn_02x02_Counter_Clockwise" H 8750 3676 50  0000 C CNN
+F 2 "Connector_PinHeader_2.54mm:PinHeader_2x02_P2.54mm_Vertical_SMD" H 8700 3550 50  0001 C CNN
+F 3 "~" H 8700 3550 50  0001 C CNN
+	1    8700 3550
 	1    0    0    -1
 $EndComp
 Text Label 2650 3100 0    50   ~ 0
 PD0
-Text Label 9900 5200 0    50   ~ 0
+Text Label 9100 3650 0    50   ~ 0
 PD0
 $Comp
 L power:+5V #PWR0112
 U 1 1 6140FFCF
-P 9200 5100
-F 0 "#PWR0112" H 9200 4950 50  0001 C CNN
-F 1 "+5V" V 9215 5228 50  0000 L CNN
-F 2 "" H 9200 5100 50  0001 C CNN
-F 3 "" H 9200 5100 50  0001 C CNN
-	1    9200 5100
+P 8400 3550
+F 0 "#PWR0112" H 8400 3400 50  0001 C CNN
+F 1 "+5V" V 8415 3678 50  0000 L CNN
+F 2 "" H 8400 3550 50  0001 C CNN
+F 3 "" H 8400 3550 50  0001 C CNN
+	1    8400 3550
 	0    -1   -1   0
 $EndComp
@@
 L power:GND #PWR0113
 U 1 1 614106F8
-P 9200 5300
-F 0 "#PWR0113" H 9200 5050 50  0001 C CNN
-F 1 "GND" H 9205 5127 50  0000 C CNN
-F 2 "" H 9200 5300 50  0001 C CNN
-F 3 "" H 9200 5300 50  0001 C CNN
-	1    9200 5300
-	1    0    0    -1
-$EndComp
-Wire Wire Line
-	9900 5200 9800 5200
-Wire Wire Line
-	9300 5100 9200 5100
-Wire Wire Line
-	9200 5300 9200 5200
-Wire Wire Line
-	9200 5200 9300 5200
+P 8400 3750
+F 0 "#PWR0113" H 8400 3500 50  0001 C CNN
+F 1 "GND" H 8405 3577 50  0000 C CNN
+F 2 "" H 8400 3750 50  0001 C CNN
+F 3 "" H 8400 3750 50  0001 C CNN
+	1    8400 3750
+	1    0    0    -1
+$EndComp
+Wire Wire Line
+	9100 3650 9000 3650
+Wire Wire Line
+	8500 3550 8400 3550
+Wire Wire Line
+	8400 3750 8400 3650
+Wire Wire Line
+	8400 3650 8500 3650
 $Comp
 L symbols:TLSM U4
 U 1 1 61493463
-P 5600 1500
-F 0 "U4" H 5625 2115 50  0000 C CNN
-F 1 "TLSM" H 5625 2024 50  0000 C CNN
-F 2 "footprints:TLSM" H 5600 1500 50  0001 C CNN
-F 3 "" H 5600 1500 50  0001 C CNN
-	1    5600 1500
-	1    0    0    -1
-$EndComp
-Text Label 4950 1850 2    50   ~ 0
+P 4100 1300
+F 0 "U4" H 4100 1150 50  0000 C CNN
+F 1 "TLSM" H 4100 1500 50  0000 C CNN
+F 2 "footprints:TLSM" H 4100 1300 50  0001 C CNN
+F 3 "" H 4100 1300 50  0001 C CNN
+	1    4100 1300
+	1    0    0    -1
+$EndComp
+Text Label 3650 1400 2    50   ~ 0
 RESET
 $Comp
 L power:GND #PWR0118
 U 1 1 6149B54A
-P 6400 1300
-F 0 "#PWR0118" H 6400 1050 50  0001 C CNN
-F 1 "GND" H 6405 1127 50  0000 C CNN
-F 2 "" H 6400 1300 50  0001 C CNN
-F 3 "" H 6400 1300 50  0001 C CNN
-	1    6400 1300
-	1    0    0    -1
-$EndComp
-Wire Wire Line
-	6300 1200 6400 1200
-Wire Wire Line
-	6400 1200 6400 1300
+P 4550 1150
+F 0 "#PWR0118" H 4550 900 50  0001 C CNN
+F 1 "GND" H 4555 977 50  0000 C CNN
+F 2 "" H 4550 1150 50  0001 C CNN
+F 3 "" H 4550 1150 50  0001 C CNN
+	1    4550 1150
+	0    -1   -1   0
+$EndComp
 $Comp
 L power:GND #PWR0119
 U 1 1 6149DF29
-P 4850 1300
-F 0 "#PWR0119" H 4850 1050 50  0001 C CNN
-F 1 "GND" H 4855 1127 50  0000 C CNN
-F 2 "" H 4850 1300 50  0001 C CNN
-F 3 "" H 4850 1300 50  0001 C CNN
-	1    4850 1300
-	1    0    0    -1
-$EndComp
-Wire Wire Line
-	4850 1300 4850 1200
-Wire Wire Line
-	4850 1200 4950 1200
+P 3650 1150
+F 0 "#PWR0119" H 3650 900 50  0001 C CNN
+F 1 "GND" H 3655 977 50  0000 C CNN
+F 2 "" H 3650 1150 50  0001 C CNN
+F 3 "" H 3650 1150 50  0001 C CNN
+	1    3650 1150
+	0    1    1    0
+$EndComp
+Wire Wire Line
+	3750 1400 3650 1400
+Wire Wire Line
+	3650 1150 3750 1150
+Wire Wire Line
+	4450 1150 4550 1150
 $EndSCHEMATC

Commit message: made pcb bigger
Parts:
- C1: value C -> 0.1u
- C2, C3: value C -> 22p
- R3, R6: value R -> 75
- Y1: value Crystal -> 16MHz
Changed lines of the file:
@@
 P 5250 6500
 F 0 "R3" H 5320 6546 50  0000 L CNN
-F 1 "R" H 5320 6455 50  0000 L CNN
+F 1 "75" H 5320 6455 50  0000 L CNN
 F 2 "Resistor_SMD:R_1206_3216Metric_Pad1.30x1.75mm_HandSolder" V 5180 6500 50  0001 C CNN
 F 3 "~" H 5250 6500 50  0001 C CNN
@@
 P 5800 6500
 F 0 "R6" H 5870 6546 50  0000 L CNN
-F 1 "R" H 5870 6455 50  0000 L CNN
+F 1 "75" H 5870 6455 50  0000 L CNN
 F 2 "Resistor_SMD:R_1206_3216Metric_Pad1.30x1.75mm_HandSolder" V 5730 6500 50  0001 C CNN
 F 3 "~" H 5800 6500 50  0001 C CNN
@@
 P 4400 3550
 F 0 "Y1" H 4400 3818 50  0000 C CNN
-F 1 "Crystal" H 4400 3727 50  0000 C CNN
+F 1 "16MHz" H 4400 3727 50  0000 C CNN
 F 2 "Crystal:Crystal_HC49-4H_Vertical" H 4400 3550 50  0001 C CNN
 F 3 "~" H 4400 3550 50  0001 C CNN
@@
 P 4150 3800
 F 0 "C2" H 4265 3846 50  0000 L CNN
-F 1 "C" H 4265 3755 50  0000 L CNN
+F 1 "22p" H 4265 3755 50  0000 L CNN
 F 2 "Capacitor_SMD:C_1206_3216Metric_Pad1.33x1.80mm_HandSolder" H 4188 3650 50  0001 C CNN
 F 3 "~" H 4150 3800 50  0001 C CNN
@@
 P 4650 3800
 F 0 "C3" H 4765 3846 50  0000 L CNN
-F 1 "C" H 4765 3755 50  0000 L CNN
+F 1 "22p" H 4765 3755 50  0000 L CNN
 F 2 "Capacitor_SMD:C_1206_3216Metric_Pad1.33x1.80mm_HandSolder" H 4688 3650 50  0001 C CNN
 F 3 "~" H 4650 3800 50  0001 C CNN
@@
 P 1100 1150
 F 0 "C1" H 1215 1196 50  0000 L CNN
-F 1 "C" H 1215 1105 50  0000 L CNN
+F 1 "0.1u" H 1215 1105 50  0000 L CNN
 F 2 "Capacitor_SMD:C_1206_3216Metric_Pad1.33x1.80mm_HandSolder" H 1138 1000 50  0001 C CNN
 F 3 "~" H 1100 1150 50  0001 C CNN

Commit message: started v1.1
Parts:
- removed D11, D14: BACKLIGHT, LED_SMD:LED_1206_3216Metric_Pad1.42x1.75mm_HandSolder, symbol Device:LED
- removed J3: Conn_02x02_Counter_Clockwise, Connector_PinHeader_2.54mm:PinHeader_2x02_P2.54mm_Vertical_SMD, symbol Connector_Generic:Conn_02x02_Counter_Clockwise
- removed R6: 75, Resistor_SMD:R_1206_3216Metric_Pad1.30x1.75mm_HandSolder, symbol Device:R
- removed U4: TLSM, footprints:TLSM, symbol symbols:TLSM
- added BT1: Battery_Cell, footprints:CR1220, symbol Device:Battery_Cell
- added C5: 100n, Capacitor_SMD:C_1206_3216Metric_Pad1.33x1.80mm_HandSolder, symbol Device:C
- added D10, D11, D12, D13, D14, D9: WS2812B, LED_SMD:LED_WS2812B_PLCC4_5.0x5.0mm_P3.2mm, symbol LED:WS2812B
- added D15, D16: D, Diode_SMD:D_1206_3216Metric_Pad1.42x1.75mm_HandSolder, symbol Device:D
- added R1: 10k, Resistor_SMD:R_1206_3216Metric_Pad1.30x1.75mm_HandSolder, symbol Device:R
- added R2: R, Resistor_SMD:R_1206_3216Metric_Pad1.30x1.75mm_HandSolder, symbol Device:R
- added SW1: SW_MEC_5E, footprints:TS_1187A, symbol Switch:SW_MEC_5E
- added U4: PCF8563T, Package_SO:SOIC-8_3.9x4.9mm_P1.27mm, symbol Timer_RTC:PCF8563T
- added Y2: Crystal, Crystal:Crystal_SMD_EuroQuartz_EQ161-2Pin_3.2x1.5mm_HandSoldering, symbol Device:Crystal
- J2: footprint Connector_PinHeader_2.54mm:PinHeader_2x06_P2.54mm_Vertical_SMD -> Connector_PinSocket_2.54mm:PinSocket_2x06_P2.54mm_Vertical
- R3: value 75 -> 10k
Connections:
- net +5V: now also R3.2, C5.1, D10.1 (VDD), D11.1 (VDD), D12.1 (VDD), D13.1 (VDD), D14.1 (VDD), D15.2 (A), D9.1 (VDD), R1.1; no longer U2.16 (VLCD)
- net GND: now also BT1.2 (-), C5.2, D10.3 (VSS), D11.3 (VSS), D12.3 (VSS), D13.3 (VSS), D14.3 (VSS), D9.3 (VSS), R2.2, SW1.3 (K), SW1.4 (A), U4.4 (VSS); no longer R3.2
- net PD1: now also R3.1, SW1.1, SW1.2
- net PB1: now reaches U1.13 (PB1)
- net PB2: now reaches U1.14 (PB2)
- net PB2: now also D9.4 (DIN)
- net PC5: now reaches U1.28 (PC5)
- net PC5: now also U4.6 (SCL)
- net BACKLIGHT_LED renamed PC4
- net PC4: now also U4.5 (SDA)
- new net: R1.2, U2.16 (VLCD)
- new net: D10.4 (DIN), D9.2 (DOUT)
- new net: D10.2 (DOUT), D11.4 (DIN)
- new net: D11.2 (DOUT), D12.4 (DIN)
- new net: D12.2 (DOUT), D13.4 (DIN)
- new net: D13.2 (DOUT), D14.4 (DIN)
- new net: U4.1 (OSCI), Y2.1
- new net: U4.2 (OSCO), Y2.2
- new net: R2.1, U4.3 (~INT~)
- new net: D15.1 (K), D16.1 (K), U4.8 (VDD)
- new net: BT1.1 (+), D16.2 (A)
Other:
- note added: "Mode button"
- note removed: "LCD Backlight"
- moved on the sheet: C4, J2, U2
