File: pcb-main/pcb-main.sch (KiCad schematic (older format))
At the start: 36 parts, among them J1 AVR-ISP-6, J2 Conn_02x06_Counter_Clockwise, M1 Stepper_Motor, SW1 SW_MEC_5E, U1 ATmega328P-AU, U2 HT1621B, U3 VIM878, U4 PCF8563T, Y1 16MHz, Y2 Crystal

Commit message: v1.1
Parts:
- C1: value 0.1u -> 100n
- C4: value C -> 100n
- D10, D11, D12, D13, D14, D9: LCSC (none) -> C2761795
- D15, D16: value D -> 1N4001
- R2: value R -> 10k
- SW1: LCSC (none) -> C318884
- U1: LCSC (none) -> C14877
- U2: value HT1621B -> HT1621B-LQFP-A; footprint footprints:HT1621B -> Package_QFP:LQFP-48_7x7mm_P0.5mm; symbol symbols:HT1621B -> symbols:HT1621B-LQFP-A; LCSC (none) -> C7532
- U4: LCSC (none) -> C7440
- Y2: value Crystal -> 32kHz; footprint Crystal:Crystal_SMD_EuroQuartz_EQ161-2Pin_3.2x1.5mm_HandSoldering -> Crystal:Crystal_C26-LF_D2.1mm_L6.5mm_Horizontal
Connections:
- net +5V: now also U2.9 (VDD); no longer C5.1, U2.17 (VDD)
- net COM0: now also U2.13 (COM0); no longer U2.21 (COM0)
- net COM1: now also U2.14 (COM1); no longer U2.22 (COM1)
- net COM2: now also U2.15 (COM2), U3.19 (COM2); no longer U2.23 (COM2), U3.20 (COM3)
- net COM3: now also U2.16 (COM3), U3.20 (COM3); no longer U2.24 (COM3), U3.19 (COM2)
- net GND: now also U2.5 (VSS); no longer U2.13 (VSS)
- net PB3: now also U2.4 (DATA); no longer U2.9 (CS)
- net PB4: now also U2.3 (WR); no longer U2.11 (WR)
- net PB5: now also U2.1 (CS); no longer U2.12 (DATA)
- net SEG0: now also U2.48 (SEG0), U3.36; no longer U2.8 (SEG0), U3.16 (8L)
- net SEG1: now also U2.47 (SEG1), U3.35; no longer U2.7 (SEG1), U3.15 (8D)
- net SEG10: now also U2.38 (SEG10), U3.26 (6M); no longer U2.46 (SEG10), U3.3 (2D)
- net SEG11: now also U2.37 (SEG11), U3.25 (DP6); no longer U2.45 (SEG11), U3.4 (2L)
- net SEG12: now also U2.36 (SEG12), U3.24 (7M); no longer U2.44 (SEG12), U3.5 (3D)
- net SEG13: now also U2.35 (SEG13), U3.23 (DP7); no longer U2.43 (SEG13), U3.6 (3L)
- net SEG14: now also U2.34 (SEG14), U3.22 (8M); no longer U2.42 (SEG14), U3.7 (4D)
- net SEG15: now also U2.33 (SEG15), U3.21 (DP8); no longer U2.41 (SEG15), U3.8 (4L)
- net SEG16: now also U2.32 (SEG16), U3.16 (8L); no longer U2.40 (SEG16), U3.36
- net SEG17: now also U2.31 (SEG17), U3.15 (8D); no longer U2.39 (SEG17), U3.35
- net SEG18: now also U2.30 (SEG18), U3.14 (7L); no longer U2.38 (SEG18), U3.34 (2M)
- net SEG19: now also U2.29 (SEG19), U3.13 (7D); no longer U2.37 (SEG19), U3.33 (DP2)
- net SEG2: now also U2.46 (SEG2), U3.34 (2M); no longer U2.6 (SEG2), U3.14 (7L)
- net SEG20: now also U2.28 (SEG20), U3.12 (6L); no longer U2.36 (SEG20), U3.32 (3M)
- net SEG21: now also U2.27 (SEG21), U3.11 (6D); no longer U2.35 (SEG21), U3.31 (DP3)
- net SEG22: now also U2.26 (SEG22), U3.10 (5L); no longer U2.34 (SEG22), U3.30 (4M)
- net SEG23: now also U2.25 (SEG23), U3.9 (5D); no longer U2.33 (SEG23), U3.29 (DP4)
- net SEG24: now also U2.24 (SEG24), U3.8 (4L); no longer U2.32 (SEG24), U3.28 (5M)
- net SEG25: now also U2.23 (SEG25), U3.7 (4D); no longer U2.31 (SEG25), U3.27 (DP5)
- net SEG26: now also U2.22 (SEG26), U3.6 (3L); no longer U2.30 (SEG26), U3.26 (6M)
- net SEG27: now also U2.20 (SEG27), U3.4 (2L); no longer U2.29 (SEG27), U3.25 (DP6)
- net SEG28: now also U2.21 (SEG28), U3.5 (3D); no longer U2.28 (SEG28), U3.24 (7M)
- net SEG29: now also U2.19 (SEG29), U3.3 (2D); no longer U2.27 (SEG29), U3.23 (DP7)
- net SEG3: now also U2.45 (SEG3), U3.33 (DP2); no longer U2.5 (SEG3), U3.13 (7D)
- net SEG30: now also U2.18 (SEG30), U3.2 (1L); no longer U2.26 (SEG30), U3.22 (8M)
- net SEG31: now also U2.17 (SEG31), U3.1 (1D); no longer U2.25 (SEG31), U3.21 (DP8)
- net SEG4: now also U2.44 (SEG4), U3.32 (3M); no longer U2.4 (SEG4), U3.12 (6L)
- net SEG5: now also U2.43 (SEG5), U3.31 (DP3); no longer U2.3 (SEG5), U3.11 (6D)
- net SEG6: now also U2.42 (SEG6), U3.30 (4M); no longer U2.2 (SEG6), U3.10 (5L)
- net SEG7: now also U2.41 (SEG7), U3.29 (DP4); no longer U2.1 (SEG7), U3.9 (5D)
- net SEG8: now also U2.40 (SEG8), U3.28 (5M); no longer U2.48 (SEG8), U3.1 (1D)
- net SEG9: now also U2.39 (SEG9), U3.27 (DP5); no longer U2.47 (SEG9), U3.2 (1L)
- net at R1.2: now also U2.8 (VLCD); no longer U2.16 (VLCD)
- net at D15.1 (K), D16.1 (K), U4.8 (VDD): now also C5.1
Other:
- moved on the sheet: C4, C5, R1, U2, U3
