File: pcb-main/pcb-main.kicad_sch (KiCad schematic)
At the start: 36 parts, among them J1 AVR-ISP-6, J2 Conn_02x06_Counter_Clockwise, M1 Stepper_Motor, SW1 SW_MEC_5E, U1 ATmega328P-AU, U2 HT1621B-LQFP-A, U3 VIM878, U4 PCF8563T, Y1 16MHz, Y2 32kHz

Commit message: clean up
Connections:
- net MOT_1 renamed PC1
- net MOT_2 renamed PC0
- net MOT_3 renamed PC3
- net MOT_4 renamed PC2
Changed lines of the file:
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@@
     (effects (font (size 1.27 1.27)) (justify left bottom))
   )
-  (label "MOT_4" (at 67.31 63.5 0)
+  (label "PC2" (at 67.31 63.5 0)
     (effects (font (size 1.27 1.27)) (justify left bottom))
   )
@@
     (effects (font (size 1.27 1.27)) (justify left bottom))
   )
-  (label "MOT_3" (at 67.31 66.04 0)
+  (label "PC3" (at 67.31 66.04 0)
     (effects (font (size 1.27 1.27)) (justify left bottom))
   )
@@
     (effects (font (size 1.27 1.27)) (justify right bottom))
   )
-  (label "MOT_1" (at 275.59 36.83 0)
+  (label "PC1" (at 275.59 36.83 0)
     (effects (font (size 1.27 1.27)) (justify left bottom))
   )
@@
     (effects (font (size 1.27 1.27)) (justify right bottom))
   )
-  (label "MOT_1" (at 67.31 60.96 0)
+  (label "PC1" (at 67.31 60.96 0)
     (effects (font (size 1.27 1.27)) (justify left bottom))
   )
@@
     (effects (font (size 1.27 1.27)) (justify left bottom))
   )
-  (label "MOT_4" (at 214.63 50.8 180)
+  (label "PC2" (at 214.63 50.8 180)
     (effects (font (size 1.27 1.27)) (justify right bottom))
   )
@@
     (effects (font (size 1.27 1.27)) (justify left bottom))
   )
-  (label "MOT_2" (at 67.31 58.42 0)
+  (label "PC0" (at 67.31 58.42 0)
     (effects (font (size 1.27 1.27)) (justify left bottom))
   )
@@
     (effects (font (size 1.27 1.27)) (justify left bottom))
   )
-  (label "MOT_2" (at 275.59 39.37 0)
+  (label "PC0" (at 275.59 39.37 0)
     (effects (font (size 1.27 1.27)) (justify left bottom))
   )
@@
     (effects (font (size 1.27 1.27)) (justify left bottom))
   )
-  (label "MOT_3" (at 214.63 45.72 180)
+  (label "PC3" (at 214.63 45.72 180)
     (effects (font (size 1.27 1.27)) (justify right bottom))
   )
@@
     (effects (font (size 1.27 1.27)) (justify left bottom))
   )
-  (symbol (lib_id "Motor:Stepper_Motor_bipolar") (at 242.57 48.26 0)
+  (symbol (lib_id "Motor:Stepper_Motor_bipolar") (at 242.57 48.26 0) (unit 1)
     (in_bom yes) (on_board yes)
     (property "Reference" "M1" (id 0) (at 247.3452 45.1104 0)
@@
     (pin "4")
   )
-  (symbol (lib_id "Diode:1N4001") (at 217.17 57.15 270)
+  (symbol (lib_id "Diode:1N4001") (at 217.17 57.15 270) (unit 1)
     (in_bom yes) (on_board yes)
     (property "Reference" "D2" (id 0) (at 222.6818 57.15 0))
@@
     (pin "2")
   )
-  (symbol (lib_id "Diode:1N4001") (at 227.33 57.15 270)
+  (symbol (lib_id "Diode:1N4001") (at 227.33 57.15 270) (unit 1)
     (in_bom yes) (on_board yes)
     (property "Reference" "D4" (id 0) (at 232.8418 57.15 0))
@@
     (pin "2")
   )
-  (symbol (lib_id "Diode:1N4001") (at 217.17 30.48 270)
+  (symbol (lib_id "Diode:1N4001") (at 217.17 30.48 270) (unit 1)
     (in_bom yes) (on_board yes)
     (property "Reference" "D1" (id 0) (at 222.6818 30.48 0))
@@
     (pin "2")
   )
-  (symbol (lib_id "Diode:1N4001") (at 227.33 30.48 270)
+  (symbol (lib_id "Diode:1N4001") (at 227.33 30.48 270) (unit 1)
     (in_bom yes) (on_board yes)
     (property "Reference" "D3" (id 0) (at 232.8418 30.48 0))
@@
     (pin "2")
   )
-  (symbol (lib_id "Diode:1N4001") (at 262.89 57.15 270)
+  (symbol (lib_id "Diode:1N4001") (at 262.89 57.15 270) (unit 1)
     (in_bom yes) (on_board yes)
     (property "Reference" "D6" (id 0) (at 268.4018 57.15 0))
@@
     (pin "2")
   )
-  (symbol (lib_id "Diode:1N4001") (at 262.89 30.48 270)
+  (symbol (lib_id "Diode:1N4001") (at 262.89 30.48 270) (unit 1)
     (in_bom yes) (on_board yes)
     (property "Reference" "D5" (id 0) (at 268.4018 30.48 0))
@@
     (pin "2")
   )
-  (symbol (lib_id "Diode:1N4001") (at 273.05 30.48 270)
+  (symbol (lib_id "Diode:1N4001") (at 273.05 30.48 270) (unit 1)
     (in_bom yes) (on_board yes)
     (property "Reference" "D7" (id 0) (at 278.5618 30.48 0))
@@
     (pin "2")
   )
-  (symbol (lib_id "Diode:1N4001") (at 273.05 57.15 270)
+  (symbol (lib_id "Diode:1N4001") (at 273.05 57.15 270) (unit 1)
     (in_bom yes) (on_board yes)
     (property "Reference" "D8" (id 0) (at 278.5618 57.15 0))
@@
     (pin "2")
   )
-  (symbol (lib_id "power:GND") (at 217.17 66.04 0)
+  (symbol (lib_id "power:GND") (at 217.17 66.04 0) (unit 1)
     (in_bom yes) (on_board yes)
     (property "Reference" "#PWR0101" (id 0) (at 217.17 72.39 0)
@@
     (pin "1")
   )
-  (symbol (lib_id "power:+5V") (at 217.17 21.59 0)
+  (symbol (lib_id "power:+5V") (at 217.17 21.59 0) (unit 1)
     (in_bom yes) (on_board yes)
     (property "Reference" "#PWR0102" (id 0) (at 217.17 25.4 0)
@@
     (pin "1")
   )
-  (symbol (lib_id "MCU_Microchip_ATmega:ATmega328P-AU") (at 52.07 66.04 0)
+  (symbol (lib_id "MCU_Microchip_ATmega:ATmega328P-AU") (at 52.07 66.04 0) (unit 1)
     (in_bom yes) (on_board yes)
     (property "Reference" "U1" (id 0) (at 50.8 87.63 0))
@@
     (pin "9")
   )
-  (symbol (lib_id "power:+5V") (at 54.61 22.86 0)
+  (symbol (lib_id "power:+5V") (at 54.61 22.86 0) (unit 1)
     (in_bom yes) (on_board yes)
     (property "Reference" "#PWR0103" (id 0) (at 54.61 26.67 0)
@@
     (pin "1")
   )
-  (symbol (lib_id "power:+5V") (at 151.13 25.4 0)
+  (symbol (lib_id "power:+5V") (at 151.13 25.4 0) (unit 1)
     (in_bom yes) (on_board yes)
     (property "Reference" "#PWR0104" (id 0) (at 151.13 29.21 0)
@@
     (pin "1")
   )
-  (symbol (lib_id "power:GND") (at 151.13 53.34 0)
+  (symbol (lib_id "power:GND") (at 151.13 53.34 0) (unit 1)
     (in_bom yes) (on_board yes)
     (property "Reference" "#PWR0105" (id 0) (at 151.13 59.69 0)
@@
     (pin "1")
   )
-  (symbol (lib_id "Connector:AVR-ISP-6") (at 153.67 40.64 0)
+  (symbol (lib_id "Connector:AVR-ISP-6") (at 153.67 40.64 0) (unit 1)
     (in_bom yes) (on_board yes)
     (property "Reference" "J1" (id 0) (at 145.3134 38.2016 0)
@@
     (pin "1")
   )
-  (symbol (lib_id "power:+5V") (at 82.55 60.96 0)
+  (symbol (lib_id "power:+5V") (at 82.55 60.96 0) (unit 1)
     (in_bom yes) (on_board yes)
     (property "Reference" "#PWR0114" (id 0) (at 82.55 64.77 0)
@@
     (pin "2")
   )
-  (symbol (lib_id "power:GND") (at 105.41 105.41 0)
+  (symbol (lib_id "power:GND") (at 105.41 105.41 0) (unit 1)
     (in_bom yes) (on_board yes)
     (property "Reference" "#PWR0111" (id 0) (at 105.41 111.76 0)
@@
     (pin "2")
   )
-  (symbol (lib_id "power:GND") (at 27.94 33.02 0)
+  (symbol (lib_id "power:GND") (at 27.94 33.02 0) (unit 1)
     (in_bom yes) (on_board yes)
     (property "Reference" "#PWR0115" (id 0) (at 27.94 39.37 0)
@@
     (pin "1")
   )
-  (symbol (lib_id "power:+5V") (at 161.29 92.71 270)
+  (symbol (lib_id "power:+5V") (at 161.29 92.71 270) (unit 1)
     (in_bom yes) (on_board yes)
     (property "Reference" "#PWR0116" (id 0) (at 157.48 92.71 0)
@@
     (pin "1")
   )
-  (symbol (lib_id "power:GND") (at 161.29 87.63 90)
+  (symbol (lib_id "power:GND") (at 161.29 87.63 90) (unit 1)
     (in_bom yes) (on_board yes)
     (property "Reference" "#PWR0117" (id 0) (at 167.64 87.63 0)
@@
     (pin "9")
   )
-  (symbol (lib_id "power:GND") (at 52.07 104.14 0)
+  (symbol (lib_id "power:GND") (at 52.07 104.14 0) (unit 1)
     (in_bom yes) (on_board yes)
     (property "Reference" "#PWR0106" (id 0) (at 52.07 110.49 0)
@@
     (pin "1")
   )
-  (symbol (lib_id "power:GND") (at 191.77 99.06 0)
+  (symbol (lib_id "power:GND") (at 191.77 99.06 0) (unit 1)
     (in_bom yes) (on_board yes)
     (property "Reference" "#PWR0123" (id 0) (at 191.77 105.41 0)
@@
     (pin "1")
   )
-  (symbol (lib_id "power:GND") (at 207.01 99.06 0)
+  (symbol (lib_id "power:GND") (at 207.01 99.06 0) (unit 1)
     (in_bom yes) (on_board yes)
     (property "Reference" "#PWR0124" (id 0) (at 207.01 105.41 0)
@@
     (pin "1")
   )
-  (symbol (lib_id "power:GND") (at 222.25 99.06 0)
+  (symbol (lib_id "power:GND") (at 222.25 99.06 0) (unit 1)
     (in_bom yes) (on_board yes)
     (property "Reference" "#PWR0125" (id 0) (at 222.25 105.41 0)
@@
     (pin "1")
   )
-  (symbol (lib_id "power:GND") (at 237.49 99.06 0)
+  (symbol (lib_id "power:GND") (at 237.49 99.06 0) (unit 1)
     (in_bom yes) (on_board yes)
     (property "Reference" "#PWR0126" (id 0) (at 237.49 105.41 0)
@@
     (pin "1")
   )
-  (symbol (lib_id "power:GND") (at 252.73 99.06 0)
+  (symbol (lib_id "power:GND") (at 252.73 99.06 0) (unit 1)
     (in_bom yes) (on_board yes)
     (property "Reference" "#PWR0127" (id 0) (at 252.73 105.41 0)
@@
     (pin "1")
   )
-  (symbol (lib_id "power:GND") (at 267.97 99.06 0)
+  (symbol (lib_id "power:GND") (at 267.97 99.06 0) (unit 1)
     (in_bom yes) (on_board yes)
     (property "Reference" "#PWR0128" (id 0) (at 267.97 105.41 0)
@@
     (pin "1")
   )
-  (symbol (lib_id "power:GND") (at 217.17 151.13 0)
+  (symbol (lib_id "power:GND") (at 217.17 151.13 0) (unit 1)
     (in_bom yes) (on_board yes)
     (property "Reference" "#PWR0119" (id 0) (at 217.17 157.48 0)
@@
     (pin "2")
   )
-  (symbol (lib_id "power:GND") (at 229.87 158.75 0)
+  (symbol (lib_id "power:GND") (at 229.87 158.75 0) (unit 1)
     (in_bom yes) (on_board yes)
     (property "Reference" "#PWR0129" (id 0) (at 229.87 165.1 0)
@@
     (pin "2")
   )
-  (symbol (lib_id "power:GND") (at 238.76 135.89 0)
+  (symbol (lib_id "power:GND") (at 238.76 135.89 0) (unit 1)
     (in_bom yes) (on_board yes)
     (property "Reference" "#PWR0130" (id 0) (at 238.76 142.24 0)
@@
     (pin "2")
   )
-  (symbol (lib_id "power:GND") (at 185.42 134.62 0)
+  (symbol (lib_id "power:GND") (at 185.42 134.62 0) (unit 1)
     (in_bom yes) (on_board yes)
     (property "Reference" "#PWR0131" (id 0) (at 185.42 140.97 0)
@@
     (pin "2")
   )
-  (symbol (lib_id "power:+5V") (at 102.87 21.59 0)
+  (symbol (lib_id "power:+5V") (at 102.87 21.59 0) (unit 1)
     (in_bom yes) (on_board yes)
     (property "Reference" "#PWR0132" (id 0) (at 102.87 25.4 0)
@@
     (pin "1")
   )
-  (symbol (lib_id "power:GND") (at 118.11 39.37 0)
+  (symbol (lib_id "power:GND") (at 118.11 39.37 0) (unit 1)
     (in_bom yes) (on_board yes)
     (property "Reference" "#PWR0133" (id 0) (at 118.11 45.72 0)
