File: pcb-main/pcb-main.kicad_sch (KiCad schematic)
At the start: 43 parts, among them J1 AVR-ISP-6, J2 Conn_02x06_Counter_Clockwise, M1 Stepper_Motor, SW1 SW_MEC_5E, SW2 SW_MEC_5E, U1 ATmega328P-AU, U2 HT1621B-LQFP-A, U3 VIM878, U4 PCF8563T, Y1 Crystal_GND24, Y2 32kHz

Commit message: update layout
Parts:
- removed SW1, SW2: SW_MEC_5E, footprints:TS_1187A, symbol Switch:SW_MEC_5E
- added J3: Conn_01x02_Male, Connector_JST:JST_PH_S2B-PH-K_1x02_P2.00mm_Horizontal, symbol Connector:Conn_01x02_Male
- added SW1: SW_Push, Button_Switch_SMD:SW_SPST_TL3342, symbol Switch:SW_Push
- C1, C2, C3, C4, C5: footprint Capacitor_SMD:C_1206_3216Metric_Pad1.33x1.80mm_HandSolder -> Capacitor_SMD:C_0805_2012Metric
- D15, D16: footprint Diode_SMD:D_1206_3216Metric_Pad1.42x1.75mm_HandSolder -> Diode_SMD:D_0805_2012Metric
- J2: footprint Connector_PinSocket_2.54mm:PinSocket_2x06_P2.54mm_Vertical -> Connector_PinHeader_2.00mm:PinHeader_2x06_P2.00mm_Vertical
- R1, R2, R3, R7: footprint Resistor_SMD:R_1206_3216Metric_Pad1.30x1.75mm_HandSolder -> Resistor_SMD:R_0805_2012Metric
Connections:
- net GND: now also J3.1 (Pin_1), SW1.2
- net PD0: now also R3.1, J3.2 (Pin_2)
- net PD1: no longer R3.1
- net RESET: now also SW1.1
Other:
- note added: "Board to board connector"
- note added: "Crystal oscillator"
- note added: "ICSP"
- note added: "Neopixels"
- note added: "Real time clock"
- note added: "Stepper motor"
- note removed: "ISP"
- moved on the sheet: BT1, C2, C3, C5, D15, D16, J1, J2, R2, R3, R7, Y1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

Commit message: update pcb layouts
Parts:
- M1: footprint footprints:Stepper Motor -> footprints:X27.168
Other:
- moved on the sheet: J1, J2, J3, R3

Commit message: v1.3 last minute changes
Parts:
- C1, C10, C11, C4, C5, C6, C7, C8, C9: LCSC (none) -> C49678
- C2, C3: JLCPCB (none) -> (none); LCSC (none) -> C1804
- D15, D16: value 1N4001 -> 1N5819WS; footprint Diode_SMD:D_0805_2012Metric -> Diode_SMD:D_SOD-323; LCSC (none) -> C191023
- R1: LCSC (none) -> C149504
- R2, R3, R7: LCSC (none) -> C17414
- SW1: LCSC (none) -> C318884
- Y1: value Crystal_GND24 -> X322516MLB4SI; LCSC (none) -> C13738
- Y2: value 32kHz -> Q13FC1350000400; LCSC (none) -> C32346
