File: pcb-sensor/pcb-sensor.sch (KiCad schematic (older format))
At the start: 20 parts, among them J1 Conn_02x06_Counter_Clockwise, J2 Conn_01x10, SW1 SW_Push, U1 LM340T-5, U2 4N35, U3 4N35, U4 4N35

Commit message: sensor pcb
Parts:
- removed J2: Conn_01x10, Connector_JST:JST_XH_S10B-XH-A_1x10_P2.50mm_Horizontal, symbol Connector_Generic:Conn_01x10
- removed SW1: SW_Push, Button_Switch_SMD:SW_DIP_SPSTx01_Slide_6.7x4.1mm_W6.73mm_P2.54mm_LowProfile_JPin, symbol Switch:SW_Push
- removed U1: LM340T-5, symbol symbols:LM340T-5
- added D3: D, Diode_SMD:D_1206_3216Metric_Pad1.42x1.75mm_HandSolder, symbol Device:D
- added J2: Conn_01x12, Connector_PinHeader_2.54mm:PinHeader_1x12_P2.54mm_Vertical, symbol Connector_Generic:Conn_01x12
- added J3: Conn_01x02, Connector_PinSocket_2.54mm:PinSocket_2x01_P2.54mm_Vertical, symbol Connector_Generic:Conn_01x02
- added R11, R12: R, Resistor_SMD:R_1206_3216Metric_Pad1.30x1.75mm_HandSolder, symbol Device:R
- added U1: LM340MP, Package_TO_SOT_SMD:SOT-223, symbol symbols:LM340MP
- added U5: TLSM, footprints:TLSM, symbol symbols:TLSM
- U2, U3, U4: footprint Package_DIP:DIP-6_W7.62mm -> footprints:4N35S
Connections:
- net PD7 is gone; now on net NEUTRAL: J1.6 (Pin_6)
- net +12V: now also J2.2 (Pin_2), U1.1 (IN)
- net +5V: now also D3.1 (K), J2.11 (Pin_11), R11.1, R12.1, U1.3 (Out)
- net ADC6: no longer C1.1, R5.2, R6.1
- net ADC7: now also C1.1, R5.2, R6.1, D3.2 (A)
- net GND: now also J2.1 (Pin_1), J2.12 (Pin_12), J3.2 (Pin_2), U1.2 (GND), U1.4 (GND), U5.1 (A)
- net KEY_12V: now also J2.3 (Pin_3)
- net PD1: now also J3.1 (Pin_1), R12.2, U5.4 (D); no longer R9.2, U3.5
- net PD5: now also R9.2, U3.5; no longer R10.2, U4.5
- net PD6: now also R10.2, U4.5
- net HIGH_BEAM_12V renamed HIGH_BEAM
- net HIGH_BEAM: now also J2.4 (Pin_4)
- net NEUTRAL_12V renamed NEUTRAL
- net NEUTRAL: now also J2.5 (Pin_5); no longer J1.5 (Pin_5)
- net TACHO_12V renamed COIL
- net COIL: now also J2.9 (Pin_9)
- net TURN_SIGNAL_LEFT_12V renamed TURN_SIGNAL_LEFT
- net TURN_SIGNAL_LEFT: now also J2.8 (Pin_8)
- net TURN_SIGNAL_RIGHT_12V renamed TURN_SIGNAL_RIGHT
- net TURN_SIGNAL_RIGHT: now also J2.7 (Pin_7)
- new net OIL_PRESSURE: J2.6 (Pin_6)
- new net PD2: J1.5 (Pin_5), J2.10 (Pin_10), R11.2
Other:
- note added: "Battery voltage"
- note added: "High beam indicator"
- note added: "Mode button"
- note added: "Neutral switch"
- note added: "Oil pressure switch"
- note added: "Power supply"
- note added: "Speedometer"
- note added: "Tachometer"
- note added: "Turn signal indicator"
- note removed: "TODO: speedo"
- moved on the sheet: C1, D1, D2, R1, R10, R2, R3, R4, R5, R6, R7, R8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

Commit message: v1.0
Connections:
- net OIL_PRESSURE_12V is gone; now on net OIL_PRESSURE: J1.3 (Pin_3), R3.2
- net +12V: now also J2.9 (Pin_9); no longer J2.2 (Pin_2)
- net COIL: now also J2.8 (Pin_8); no longer J2.9 (Pin_9)
- net HIGH_BEAM: now also J2.2 (Pin_2); no longer J2.4 (Pin_4)
- net KEY_12V: now also J2.5 (Pin_5); no longer J2.3 (Pin_3)
- net NEUTRAL: now also J2.7 (Pin_7); no longer J2.5 (Pin_5)
- net TURN_SIGNAL_LEFT: now also J2.4 (Pin_4); no longer J2.8 (Pin_8)
- net TURN_SIGNAL_RIGHT: now also J2.3 (Pin_3); no longer J2.7 (Pin_7)
Changed lines of the file:
@@
 	0    1    1    0
 $EndComp
-Text Label 2250 3400 0    50   ~ 0
+Text Label 2250 3500 0    50   ~ 0
 COIL
 Text Label 2250 3100 0    50   ~ 0
 SPEED_GND
-Text Label 2250 3500 0    50   ~ 0
+Text Label 2250 3900 0    50   ~ 0
 TURN_SIGNAL_LEFT
 Text Label 2250 3700 0    50   ~ 0
 OIL_PRESSURE
-Text Label 2250 3800 0    50   ~ 0
+Text Label 2250 3600 0    50   ~ 0
 NEUTRAL
-Text Label 2250 3900 0    50   ~ 0
+Text Label 2250 4100 0    50   ~ 0
 HIGH_BEAM
 $Comp
@@
 L power:+12V #PWR0105
 U 1 1 613DEE20
-P 2350 4100
-F 0 "#PWR0105" H 2350 3950 50  0001 C CNN
-F 1 "+12V" V 2365 4228 50  0000 L CNN
-F 2 "" H 2350 4100 50  0001 C CNN
-F 3 "" H 2350 4100 50  0001 C CNN
-	1    2350 4100
+P 2250 3400
+F 0 "#PWR0105" H 2250 3250 50  0001 C CNN
+F 1 "+12V" V 2265 3528 50  0000 L CNN
+F 2 "" H 2250 3400 50  0001 C CNN
+F 3 "" H 2250 3400 50  0001 C CNN
+	1    2250 3400
 	0    1    1    0
 $EndComp
-Wire Wire Line
-	2150 4100 2350 4100
 Wire Wire Line
 	2150 4200 2250 4200
@@
 Connection ~ 7250 1750
 Text Label 9750 1800 2    50   ~ 0
-OIL_PRESSURE_12V
+OIL_PRESSURE
 $Comp
 L Device:R R3
@@
 	1    0    0    -1
 $EndComp
-Text Label 2250 3600 0    50   ~ 0
+Text Label 2250 4000 0    50   ~ 0
 TURN_SIGNAL_RIGHT
 Text Label 9000 2750 2    50   ~ 0
@@
 Text Label 7750 5550 0    50   ~ 0
 PD5
-Text Label 2250 4000 0    50   ~ 0
+Text Label 2250 3800 0    50   ~ 0
 KEY_12V
 Text Label 6750 4950 2    50   ~ 0
@@
 Wire Wire Line
 	4500 6200 4500 6300
+Wire Wire Line
+	2150 4100 2250 4100
 $EndSCHEMATC

Commit message: started v1.1
Parts:
- removed J2: Conn_01x12, Connector_PinHeader_2.54mm:PinHeader_1x12_P2.54mm_Vertical, symbol Connector_Generic:Conn_01x12
- removed R12: R, Resistor_SMD:R_1206_3216Metric_Pad1.30x1.75mm_HandSolder, symbol Device:R
- removed U5: TLSM, footprints:TLSM, symbol symbols:TLSM
- added C2: CP, Capacitor_THT:CP_Radial_D8.0mm_P3.80mm, symbol Device:CP
- added C3: 0.22u, Capacitor_SMD:C_1206_3216Metric_Pad1.33x1.80mm_HandSolder, symbol Device:C
- added C4: 0.1u, Capacitor_SMD:C_1206_3216Metric_Pad1.33x1.80mm_HandSolder, symbol Device:C
- added D4: 1N4148, Diode_SMD:D_1206_3216Metric_Pad1.42x1.75mm_HandSolder, symbol Device:D
- added J2, J6: Conn_01x03, Connector_PinSocket_2.54mm:PinSocket_1x03_P2.54mm_Vertical, symbol Connector_Generic:Conn_01x03
- added J4: Conn_01x05, Connector_PinSocket_2.54mm:PinSocket_1x05_P2.54mm_Vertical, symbol Connector_Generic:Conn_01x05
- added J5: Conn_01x02, Connector_PinSocket_2.54mm:PinSocket_1x02_P2.54mm_Vertical, symbol Connector_Generic:Conn_01x02
- D1, D2: value D -> 1N4148
- J1: footprint Connector_PinSocket_2.54mm:PinSocket_2x06_P2.54mm_Vertical_SMD -> Connector_PinSocket_2.54mm:PinSocket_2x06_P2.54mm_Vertical
- J3: footprint Connector_PinSocket_2.54mm:PinSocket_2x01_P2.54mm_Vertical -> Connector_PinSocket_2.54mm:PinSocket_1x02_P2.54mm_Vertical
- R1, R4: value R -> 1k
- R10, R8: value R -> 200
- R2, R3: value R -> 10k
Connections:
- net KEY_12V is gone; now on net +12V: R5.1, R7.1
- net +12V: now also C2.1, C3.1, D4.1 (K)
- net +5V: now also C4.1, J2.2 (Pin_2)
- net COIL: now also J6.3 (Pin_3)
- net GND: now also J3.1 (Pin_1), C2.2, C3.2, C4.2, J2.3 (Pin_3), J5.1 (Pin_1), J6.1 (Pin_1); no longer J3.2 (Pin_2)
- net HIGH_BEAM: now also J4.1 (Pin_1)
- net NEUTRAL: now also J4.5 (Pin_5)
- net OIL_PRESSURE: now also J4.4 (Pin_4)
- net PD2: now also J2.1 (Pin_1)
- net TURN_SIGNAL_LEFT: now also J4.3 (Pin_3)
- net TURN_SIGNAL_RIGHT: now also J4.2 (Pin_2)
- net PD1 renamed MODE_BUTTON
- net MODE_BUTTON: now also J3.2 (Pin_2); no longer J3.1 (Pin_1)
- new net: D4.2 (A), J5.2 (Pin_2)
Other:
- moved on the sheet: J3

Commit message: more v1.1
Parts:
- removed J3: Conn_01x02, Connector_PinSocket_2.54mm:PinSocket_1x02_P2.54mm_Vertical, symbol Connector_Generic:Conn_01x02
- removed R7, R9: R, Resistor_SMD:R_1206_3216Metric_Pad1.30x1.75mm_HandSolder, symbol Device:R
- removed U2, U3, U4: 4N35, footprints:4N35S, symbol Isolator:4N35
- added J3, J7, J8: Conn_01x01, Connector_PinSocket_2.54mm:PinSocket_1x01_P2.54mm_Vertical, symbol Connector_Generic:Conn_01x01
- added U2, U4: SFH617A-1, Package_SO:SOP-4_4.4x2.6mm_P1.27mm, symbol Isolator:SFH617A-1
- R10, R8: value 200 -> 10k
Connections:
- net COIL is gone; now on net PD2: J6.3 (Pin_3)
- net +12V: now also J2.2 (Pin_2), J6.2 (Pin_2)
- net +5V: no longer J2.2 (Pin_2)
- net ADC6: now also J7.1 (Pin_1)
- net GND: now also U2.2, U2.3, U4.2, U4.3
- net MODE_BUTTON: now also J3.1 (Pin_1)
- net NEUTRAL: now also J1.4 (Pin_4); no longer J1.6 (Pin_6)
- net PB0: now also J8.1 (Pin_1)
- net PD2: no longer J2.1 (Pin_1), R11.2
- net PD4: now also U2.4
- net PD5: now also R10.2, U4.4
- net at R1.2: now also U4.1
- net at R4.2: now also U2.1
- removed net PD6: J1.4 (Pin_4), R10.2
- new net PD7: J1.6 (Pin_6), J2.1 (Pin_1), R11.2
Other:
- moved on the sheet: C1, C2, C3, C4, D3, D4, J2, J4, J5, J6, R10, R11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

Commit message: v1.1
Parts:
- C1: value C -> 100n
- C2: value CP -> 100u
- D1, D2, D4: value 1N4148 -> 1N4001
- D3: value D -> 1N4001
- R11, R5: value R -> 10k
- R6: value R -> 4.7k
Other:
- note added: "Black"
- note added: "Blue"
- note added: "Brown"
Changed lines of the file:
@@
 Text Label 2150 4400 0    50   ~ 0
 PD1
-Text Label 7050 1750 2    50   ~ 0
+Text Label 7150 1750 2    50   ~ 0
 NEUTRAL
 $Comp
@@
 Wire Wire Line
 	7450 1750 7250 1750
-Wire Wire Line
-	7050 1750 7250 1750
-Connection ~ 7250 1750
-Text Label 9750 1800 2    50   ~ 0
+Text Label 9850 1800 2    50   ~ 0
 OIL_PRESSURE
 $Comp
@@
 PD3
 Wire Wire Line
-	9750 1800 9950 1800
-Wire Wire Line
 	9950 1800 9950 1700
-Connection ~ 9950 1800
 Wire Wire Line
 	9950 1800 10150 1800
@@
 P 9250 2750
 F 0 "D1" H 9250 2550 50  0000 C CNN
-F 1 "1N4148" H 9250 2650 50  0000 C CNN
+F 1 "1N4001" H 9250 2650 50  0000 C CNN
 F 2 "Diode_SMD:D_1206_3216Metric_Pad1.42x1.75mm_HandSolder" H 9250 2750 50  0001 C CNN
 F 3 "~" H 9250 2750 50  0001 C CNN
@@
 P 9250 2950
 F 0 "D2" H 9250 3150 50  0000 C CNN
-F 1 "1N4148" H 9250 3050 50  0000 C CNN
+F 1 "1N4001" H 9250 3050 50  0000 C CNN
 F 2 "Diode_SMD:D_1206_3216Metric_Pad1.42x1.75mm_HandSolder" H 9250 2950 50  0001 C CNN
 F 3 "~" H 9250 2950 50  0001 C CNN
@@
 P 3800 3500
 F 0 "R5" H 3870 3546 50  0000 L CNN
-F 1 "R" H 3870 3455 50  0000 L CNN
+F 1 "10k" H 3870 3455 50  0000 L CNN
 F 2 "Resistor_SMD:R_1206_3216Metric_Pad1.30x1.75mm_HandSolder" V 3730 3500 50  0001 C CNN
 F 3 "~" H 3800 3500 50  0001 C CNN
@@
 P 3800 4000
 F 0 "R6" H 3870 4046 50  0000 L CNN
-F 1 "R" H 3870 3955 50  0000 L CNN
+F 1 "4.7k" H 3870 3955 50  0000 L CNN
 F 2 "Resistor_SMD:R_1206_3216Metric_Pad1.30x1.75mm_HandSolder" V 3730 4000 50  0001 C CNN
 F 3 "~" H 3800 4000 50  0001 C CNN
@@
 P 4200 4000
 F 0 "C1" H 4315 4046 50  0000 L CNN
-F 1 "C" H 4315 3955 50  0000 L CNN
+F 1 "100n" H 4315 3955 50  0000 L CNN
 F 2 "Capacitor_SMD:C_1206_3216Metric_Pad1.33x1.80mm_HandSolder" H 4238 3850 50  0001 C CNN
 F 3 "~" H 4200 4000 50  0001 C CNN
@@
 P 10300 5450
 F 0 "R11" H 10370 5496 50  0000 L CNN
-F 1 "R" H 10370 5405 50  0000 L CNN
+F 1 "10k" H 10370 5405 50  0000 L CNN
 F 2 "Resistor_SMD:R_1206_3216Metric_Pad1.30x1.75mm_HandSolder" V 10230 5450 50  0001 C CNN
 F 3 "~" H 10300 5450 50  0001 C CNN
@@
 P 4200 3500
 F 0 "D3" V 4154 3580 50  0000 L CNN
-F 1 "D" V 4245 3580 50  0000 L CNN
+F 1 "1N4001" V 4245 3580 50  0000 L CNN
 F 2 "Diode_SMD:D_1206_3216Metric_Pad1.42x1.75mm_HandSolder" H 4200 3500 50  0001 C CNN
 F 3 "~" H 4200 3500 50  0001 C CNN
@@
 P 2200 6200
 F 0 "D4" H 2200 6400 50  0000 C CNN
-F 1 "1N4148" H 2200 6300 50  0000 C CNN
+F 1 "1N4001" H 2200 6300 50  0000 C CNN
 F 2 "Diode_SMD:D_1206_3216Metric_Pad1.42x1.75mm_HandSolder" H 2200 6200 50  0001 C CNN
 F 3 "~" H 2200 6200 50  0001 C CNN
@@
 P 2600 6450
 F 0 "C2" H 2718 6496 50  0000 L CNN
-F 1 "CP" H 2718 6405 50  0000 L CNN
+F 1 "100u" H 2718 6405 50  0000 L CNN
 F 2 "Capacitor_THT:CP_Radial_D8.0mm_P3.80mm" H 2638 6300 50  0001 C CNN
 F 3 "~" H 2600 6450 50  0001 C CNN
@@
 Text Label 2000 3350 0    50   ~ 0
 PB0
+Text Notes 8450 5650 2    50   ~ 0
+Brown
+Text Notes 8450 5550 2    50   ~ 0
+Blue
+Text Notes 8450 5750 2    50   ~ 0
+Black
+Wire Wire Line
+	9850 1800 9950 1800
+Connection ~ 9950 1800
+Wire Wire Line
+	7150 1750 7250 1750
+Connection ~ 7250 1750
 $EndSCHEMATC
