File: pcb-face/pcb-face.kicad_pcb (KiCad board)
At the start: 2 copper layers, 86 x 86 mm, 5 parts

Commit message: resolves #22: see through indicator icons
Parts:
- added G***: LOGO, footprints:High_Beam_Flipped, B.Cu at (130.0, 105.0)
- added G***: LOGO, footprints:Neutral_Flipped, B.Cu at (170.0, 105.0)
- added REF**: LOGO, footprints:Turn_Signals, B.Cu at (130.0, 95.0)
- added REF**: LOGO, footprints:Warning, B.Cu at (170.0, 95.0)

Commit message: resolves #47: update silkscreen labels
Other:
- board text added: "Motorcycle Tacho v1.2"
- board text removed: "Motorcycle Tacho v1.1"
Changed lines of the file:
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@@
     )
+    (fp_poly (pts
+        (xy 1.672127 1.756006)
+        (xy 1.697536 1.744364)
+        (xy 1.731652 1.721575)
+        (xy 1.777369 1.684972)
+        (xy 1.837583 1.631888)
+        (xy 1.91519 1.559655)
+        (xy 2.013085 1.465608)
+        (xy 2.134163 1.347079)
+        (xy 2.281319 1.2014)
+        (xy 2.45745 1.025904)
+        (xy 2.562219 0.921208)
+        (xy 2.752493 0.730754)
+        (xy 2.911738 0.570789)
+        (xy 3.042695 0.438303)
+        (xy 3.148104 0.330287)
+        (xy 3.230704 0.243731)
+        (xy 3.293236 0.175625)
+        (xy 3.33844 0.12296)
+        (xy 3.369056 0.082726)
+        (xy 3.387825 0.051913)
+        (xy 3.397486 0.027512)
+        (xy 3.400779 0.006513)
+        (xy 3.400936 0)
+        (xy 3.399106 -0.020545)
+        (xy 3.391787 -0.043525)
+        (xy 3.376241 -0.071952)
+        (xy 3.349727 -0.108834)
+        (xy 3.309504 -0.15718)
+        (xy 3.252833 -0.220001)
+        (xy 3.176974 -0.300307)
+        (xy 3.079186 -0.401106)
+        (xy 2.956729 -0.525409)
+        (xy 2.806863 -0.676225)
+        (xy 2.626849 -0.856563)
+        (xy 2.562219 -0.921208)
+        (xy 2.36976 -1.113382)
+        (xy 2.207791 -1.274343)
+        (xy 2.073417 -1.406758)
+        (xy 1.963743 -1.513293)
+        (xy 1.875872 -1.596617)
+        (xy 1.806911 -1.659396)
+        (xy 1.753963 -1.704298)
+        (xy 1.714133 -1.733988)
+        (xy 1.684525 -1.751135)
+        (xy 1.662245 -1.758406)
+        (xy 1.652528 -1.759169)
+        (xy 1.586587 -1.748426)
+        (xy 1.540869 -1.727502)
+        (xy 1.505615 -1.690458)
+        (xy 1.480367 -1.636414)
+        (xy 1.463746 -1.558202)
+        (xy 1.454373 -1.448651)
+        (xy 1.45087 -1.300592)
+        (xy 1.450749 -1.258938)
+        (xy 1.450749 -0.951311)
+        (xy 0.24128 -0.951311)
+        (xy 0.191988 -0.888646)
+        (xy 0.178851 -0.870354)
+        (xy 0.168281 -0.849028)
+        (xy 0.159999 -0.819646)
+        (xy 0.153728 -0.777182)
+        (xy 0.149187 -0.716612)
+        (xy 0.146099 -0.632912)
+        (xy 0.145443 -0.594569)
+        (xy 0.499438 -0.594569)
+        (xy 1.080997 -0.594569)
+        (xy 1.292516 -0.59573)
+        (xy 1.464519 -0.599157)
+        (xy 1.594945 -0.604764)
+        (xy 1.681732 -0.612467)
+        (xy 1.720509 -0.620974)
+        (xy 1.772469 -0.658029)
+        (xy 1.806496 -0.718019)
+        (xy 1.825217 -0.808659)
+        (xy 1.831257 -0.937664)
+        (xy 1.831273 -0.946421)
+        (xy 1.831273 -1.129556)
+        (xy 2.396051 -0.564778)
+        (xy 2.96083 0)
+        (xy 2.396051 0.564778)
+        (xy 1.831273 1.129557)
+        (xy 1.831273 0.946422)
+        (xy 1.825884 0.814973)
+        (xy 1.807964 0.722333)
+        (xy 1.774889 0.660788)
+        (xy 1.724034 0.622622)
+        (xy 1.720509 0.620975)
+        (xy 1.674111 0.611487)
+        (xy 1.582247 0.604018)
+        (xy 1.44698 0.598655)
+        (xy 1.27037 0.595482)
+        (xy 1.080997 0.594569)
+        (xy 0.499438 0.594569)
+        (xy 0.499438 -0.594569)
+        (xy 0.145443 -0.594569)
+        (xy 0.144185 -0.521057)
+        (xy 0.143165 -0.376024)
+        (xy 0.142763 -0.192787)
+        (xy 0.142696 0)
+        (xy 0.142791 0.220262)
+        (xy 0.143262 0.397982)
+        (xy 0.144387 0.538186)
+        (xy 0.146446 0.645897)
+        (xy 0.149716 0.72614)
+        (xy 0.154476 0.78394)
+        (xy 0.161006 0.82432)
+        (xy 0.169584 0.852305)
+        (xy 0.180488 0.87292)
+        (xy 0.191988 0.888647)
+        (xy 0.24128 0.951311)
+        (xy 1.450749 0.951311)
+        (xy 1.450749 1.258939)
+        (xy 1.453974 1.429359)
+        (xy 1.465071 1.55785)
+        (xy 1.486174 1.649704)
+        (xy 1.519417 1.710209)
+        (xy 1.566933 1.744656)
+        (xy 1.630857 1.758334)
+        (xy 1.652528 1.759169)
+      ) (layer "B.Mask") (width 0) (fill solid))
     (fp_poly (pts
         (xy -1.583503 1.750473)
@@
         (xy -1.662245 1.758407)
         (xy -1.652529 1.759169)
-      ) (layer "B.Mask") (width 0) (fill solid))
-    (fp_poly (pts
-        (xy 1.672127 1.756006)
-        (xy 1.697536 1.744364)
-        (xy 1.731652 1.721575)
-        (xy 1.777369 1.684972)
-        (xy 1.837583 1.631888)
-        (xy 1.91519 1.559655)
-        (xy 2.013085 1.465608)
-        (xy 2.134163 1.347079)
-        (xy 2.281319 1.2014)
-        (xy 2.45745 1.025904)
-        (xy 2.562219 0.921208)
-        (xy 2.752493 0.730754)
-        (xy 2.911738 0.570789)
-        (xy 3.042695 0.438303)
-        (xy 3.148104 0.330287)
-        (xy 3.230704 0.243731)
-        (xy 3.293236 0.175625)
-        (xy 3.33844 0.12296)
-        (xy 3.369056 0.082726)
-        (xy 3.387825 0.051913)
-        (xy 3.397486 0.027512)
-        (xy 3.400779 0.006513)
-        (xy 3.400936 0)
-        (xy 3.399106 -0.020545)
-        (xy 3.391787 -0.043525)
-        (xy 3.376241 -0.071952)
-        (xy 3.349727 -0.108834)
-        (xy 3.309504 -0.15718)
-        (xy 3.252833 -0.220001)
-        (xy 3.176974 -0.300307)
-        (xy 3.079186 -0.401106)
-        (xy 2.956729 -0.525409)
-        (xy 2.806863 -0.676225)
-        (xy 2.626849 -0.856563)
-        (xy 2.562219 -0.921208)
-        (xy 2.36976 -1.113382)
-        (xy 2.207791 -1.274343)
-        (xy 2.073417 -1.406758)
-        (xy 1.963743 -1.513293)
-        (xy 1.875872 -1.596617)
-        (xy 1.806911 -1.659396)
-        (xy 1.753963 -1.704298)
-        (xy 1.714133 -1.733988)
-        (xy 1.684525 -1.751135)
-        (xy 1.662245 -1.758406)
-        (xy 1.652528 -1.759169)
-        (xy 1.586587 -1.748426)
-        (xy 1.540869 -1.727502)
-        (xy 1.505615 -1.690458)
-        (xy 1.480367 -1.636414)
-        (xy 1.463746 -1.558202)
-        (xy 1.454373 -1.448651)
-        (xy 1.45087 -1.300592)
-        (xy 1.450749 -1.258938)
-        (xy 1.450749 -0.951311)
-        (xy 0.24128 -0.951311)
-        (xy 0.191988 -0.888646)
-        (xy 0.178851 -0.870354)
-        (xy 0.168281 -0.849028)
-        (xy 0.159999 -0.819646)
-        (xy 0.153728 -0.777182)
-        (xy 0.149187 -0.716612)
-        (xy 0.146099 -0.632912)
-        (xy 0.145443 -0.594569)
-        (xy 0.499438 -0.594569)
-        (xy 1.080997 -0.594569)
-        (xy 1.292516 -0.59573)
-        (xy 1.464519 -0.599157)
-        (xy 1.594945 -0.604764)
-        (xy 1.681732 -0.612467)
-        (xy 1.720509 -0.620974)
-        (xy 1.772469 -0.658029)
-        (xy 1.806496 -0.718019)
-        (xy 1.825217 -0.808659)
-        (xy 1.831257 -0.937664)
-        (xy 1.831273 -0.946421)
-        (xy 1.831273 -1.129556)
-        (xy 2.396051 -0.564778)
-        (xy 2.96083 0)
-        (xy 2.396051 0.564778)
-        (xy 1.831273 1.129557)
-        (xy 1.831273 0.946422)
-        (xy 1.825884 0.814973)
-        (xy 1.807964 0.722333)
-        (xy 1.774889 0.660788)
-        (xy 1.724034 0.622622)
-        (xy 1.720509 0.620975)
-        (xy 1.674111 0.611487)
-        (xy 1.582247 0.604018)
-        (xy 1.44698 0.598655)
-        (xy 1.27037 0.595482)
-        (xy 1.080997 0.594569)
-        (xy 0.499438 0.594569)
-        (xy 0.499438 -0.594569)
-        (xy 0.145443 -0.594569)
-        (xy 0.144185 -0.521057)
-        (xy 0.143165 -0.376024)
-        (xy 0.142763 -0.192787)
-        (xy 0.142696 0)
-        (xy 0.142791 0.220262)
-        (xy 0.143262 0.397982)
-        (xy 0.144387 0.538186)
-        (xy 0.146446 0.645897)
-        (xy 0.149716 0.72614)
-        (xy 0.154476 0.78394)
-        (xy 0.161006 0.82432)
-        (xy 0.169584 0.852305)
-        (xy 0.180488 0.87292)
-        (xy 0.191988 0.888647)
-        (xy 0.24128 0.951311)
-        (xy 1.450749 0.951311)
-        (xy 1.450749 1.258939)
-        (xy 1.453974 1.429359)
-        (xy 1.465071 1.55785)
-        (xy 1.486174 1.649704)
-        (xy 1.519417 1.710209)
-        (xy 1.566933 1.744656)
-        (xy 1.630857 1.758334)
-        (xy 1.652528 1.759169)
       ) (layer "B.Mask") (width 0) (fill solid))
   )
@@
   (gr_arc (start 128 129.5) (mid 126.585786 128.914214) (end 126 127.5) (layer "Edge.Cuts") (width 0.15))
   (gr_line (start 128 129.5) (end 172 129.5) (layer "Edge.Cuts") (width 0.15))
-  (gr_text "Motorcycle Tacho\nv1.1" (at 150 82) (layer "B.SilkS")
+  (gr_text "Motorcycle Tacho\nv1.2" (at 150 82) (layer "B.SilkS")
     (effects (font (size 1 1) (thickness 0.15)) (justify mirror))
   )

Commit message: resolves #52: crystal circuit
Other:
- board text added: "Retro Gauge v1.3"
- board text removed: "Motorcycle Tacho v1.2"
Changed lines of the file:
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@@
   (gr_arc (start 128 129.5) (mid 126.585786 128.914214) (end 126 127.5) (layer "Edge.Cuts") (width 0.15))
   (gr_line (start 128 129.5) (end 172 129.5) (layer "Edge.Cuts") (width 0.15))
-  (gr_text "Motorcycle Tacho\nv1.2" (at 150 82) (layer "B.SilkS")
+  (gr_text "Retro Gauge\nv1.3" (at 150 82) (layer "B.SilkS")
     (effects (font (size 1 1) (thickness 0.15)) (justify mirror))
   )
